File: design/BQ7.sch (KiCad schematic (older format))
At the start: 41 parts

Commit message: Some small fix in BQ and TODO
Other:
- note added: "We are going to use 30 cell this is 15 so it's a half here it's a reason for this wierd BATT labels"
- note removed: "Mess bellow. Batt_ball circuit are sharing every pin expect last and first\nSo becase they are sharing pin they are sharing a Rin so only\nlast should have it.(IN every block)."
Changed lines of the file:
@@
 9F DF D1 D1 31 D6 A5 40 90 E1 4D 94 96 C0 77 F7 E1 9C E9 BB 40 B5 84 6A 00 41 90 F1 06 B5 8D 23
 08 82 20 C8 04 83 62 36 82 20 08 82 4C 0C 38 D4 12 88 20 08 82 20 E3 1C 1A 1D 89 20 08 82 20 08
-82 20 08 82 20 23 ED FF 01 11 4E 07 64 6B 3C CF 2D 00 00 00 00 49 45 4E 44 AE 42 60 82 1F
+82 20 08 82 20 23 ED FF 01 11 4E 07 64 6B 3C CF 2D 00 00 00 00 49 45 4E 44 AE 42 60 82 A5
 EndData
 $EndBitmap
@@
 $EndComp
 $Comp
-L GND #PWR?
+L GND #PWR05
 U 1 1 5584794D
 P 7300 1200
-F 0 "#PWR?" H 7300 1200 30  0001 C CNN
+F 0 "#PWR05" H 7300 1200 30  0001 C CNN
 F 1 "GND" H 7300 1130 30  0001 C CNN
 F 2 "" H 7300 1200 60  0000 C CNN
@@
 $EndComp
 $Comp
-L GND #PWR?
+L GND #PWR06
 U 1 1 55848488
 P 5700 2200
-F 0 "#PWR?" H 5700 2200 30  0001 C CNN
+F 0 "#PWR06" H 5700 2200 30  0001 C CNN
 F 1 "GND" H 5700 2130 30  0001 C CNN
 F 2 "" H 5700 2200 60  0000 C CNN
@@
 $EndComp
 $Comp
-L GND #PWR?
+L GND #PWR07
 U 1 1 5584850F
 P 5950 2200
-F 0 "#PWR?" H 5950 2200 30  0001 C CNN
+F 0 "#PWR07" H 5950 2200 30  0001 C CNN
 F 1 "GND" H 5950 2130 30  0001 C CNN
 F 2 "" H 5950 2200 60  0000 C CNN
@@
 $EndComp
 $Comp
-L GND #PWR?
+L GND #PWR08
 U 1 1 558485AD
 P 6200 2200
-F 0 "#PWR?" H 6200 2200 30  0001 C CNN
+F 0 "#PWR08" H 6200 2200 30  0001 C CNN
 F 1 "GND" H 6200 2130 30  0001 C CNN
 F 2 "" H 6200 2200 60  0000 C CNN
@@
 $EndComp
 $Comp
-L GND #PWR?
+L GND #PWR09
 U 1 1 55BCC3FD
 P 6250 5800
-F 0 "#PWR?" H 6250 5800 30  0001 C CNN
+F 0 "#PWR09" H 6250 5800 30  0001 C CNN
 F 1 "GND" H 6250 5730 30  0001 C CNN
 F 2 "" H 6250 5800 60  0000 C CNN
@@
 $EndComp
 $Comp
-L GND #PWR?
+L GND #PWR010
 U 1 1 55BCC42E
 P 7400 5800
-F 0 "#PWR?" H 7400 5800 30  0001 C CNN
+F 0 "#PWR010" H 7400 5800 30  0001 C CNN
 F 1 "GND" H 7400 5730 30  0001 C CNN
 F 2 "" H 7400 5800 60  0000 C CNN
@@
 -BATT_In
 $Comp
-L GND #PWR?
+L GND #PWR011
 U 1 1 55BCCB26
 P 6300 6550
-F 0 "#PWR?" H 6300 6550 30  0001 C CNN
+F 0 "#PWR011" H 6300 6550 30  0001 C CNN
 F 1 "GND" H 6300 6480 30  0001 C CNN
 F 2 "" H 6300 6550 60  0000 C CNN
@@
 $EndComp
 $Comp
-L GND #PWR?
+L GND #PWR012
 U 1 1 55BCD61C
 P 6550 2650
-F 0 "#PWR?" H 6550 2650 30  0001 C CNN
+F 0 "#PWR012" H 6550 2650 30  0001 C CNN
 F 1 "GND" H 6550 2580 30  0001 C CNN
 F 2 "" H 6550 2650 60  0000 C CNN
@@
 $EndComp
 $Comp
-L GND #PWR?
+L GND #PWR013
 U 1 1 55BD1E3F
 P 6950 2100
-F 0 "#PWR?" H 6950 2100 30  0001 C CNN
+F 0 "#PWR013" H 6950 2100 30  0001 C CNN
 F 1 "GND" H 6950 2030 30  0001 C CNN
 F 2 "" H 6950 2100 60  0000 C CNN
@@
 $EndComp
 $Comp
-L GND #PWR?
+L GND #PWR014
 U 1 1 55BCD4C0
 P 4750 2250
-F 0 "#PWR?" H 4750 2250 30  0001 C CNN
+F 0 "#PWR014" H 4750 2250 30  0001 C CNN
 F 1 "GND" H 4750 2180 30  0001 C CNN
 F 2 "" H 4750 2250 60  0000 C CNN
@@
 $EndComp
 $Comp
-L GND #PWR?
+L GND #PWR015
 U 1 1 55BDD023
 P 5700 1950
-F 0 "#PWR?" H 5700 1950 30  0001 C CNN
+F 0 "#PWR015" H 5700 1950 30  0001 C CNN
 F 1 "GND" H 5700 1880 30  0001 C CNN
 F 2 "" H 5700 1950 60  0000 C CNN
@@
 Text Notes 8600 5200 0    24   ~ 0
 Schottky diode for avoding high current on pin(We go to 50A+ so..)
-Text Notes 9200 0    0    39   ~ 0
-Mess bellow. Batt_ball circuit are sharing every pin expect last and first\nSo becase they are sharing pin they are sharing a Rin so only\nlast should have it.(IN every block).
 Text Notes 6050 2250 0    60   ~ 0
 This is a ground so
@@
 B
 $Comp
-L GND #PWR?
+L GND #PWR016
 U 1 1 3A4FD999
 P 11050 2700
-F 0 "#PWR?" H 11050 2700 30  0001 C CNN
+F 0 "#PWR016" H 11050 2700 30  0001 C CNN
 F 1 "GND" H 11050 2630 30  0001 C CNN
 F 2 "" H 11050 2700 60  0000 C CNN
@@
 	9400 1200 9400 2600
 Connection ~ 9400 2600
+Text Notes 6000 6100 0    20   ~ 0
+We are going to use 30 cell this is 15 so it's a half here it's a reason for this wierd BATT labels
 $EndSCHEMATC

Commit message: Renew pdf set some vaules add links and more comments
Parts:
- added C? (x2): 10u, symbol C
- C?: value 4.7u -> 12u
- C?: value C -> 4,7
- C? (x3): value Cf -> Cf 40u
- C?: value C -> 10u
- R?: value 1M -> 5M
- R?: value SHUNT -> SHUNT 10K
- R? (x2): value 100 -> 1K
Connections:
- net A: now also C?.2
- net B: now also C?.2
- net at C?.1, C?.2, R?.1: now also U?.42 (SRP)
- net at U?.11 (NC), U?.12 (NC), U?.14 (CAP2): now also C?.1
- net at U?.16 (NC), U?.17 (NC), U?.19 (CAP3): now also C?.1
Other:
- note added: "And overvoltage. They value must be very close to max batt voltage"
- note added: "And overvoltage. value must be very close to max batt voltage."
- note added: "Be caerfull with VSS and other pins beacuse we must maintaine \na specific max voltage diff between pins.\n"
- note added: "DSG CHG circuit TODO"
- note added: "Maybe to high value VSS and SRP will have to much voltage diff.\n"
- note added: "VSS basicly\n"
- moved on the sheet: C?, R?
Changed lines of the file:
@@
 $Descr A4 11693 8268
 encoding utf-8
-Sheet 3 68
+Sheet 3 101
 Title "BQ76940"
 Date ""
@@
 $Bitmap
 Pos 2300 3300
-Scale 1.000000
+Scale 1,000000
 Data
 89 50 4E 47 0D 0A 1A 0A 00 00 00 0D 49 48 44 52 00 00 04 1B 00 00 02 70 08 02 00 00 00 47 C3 FE
@@
 00 00 00 00 00 00 00 00 00 00 00 00 00 00 00 00 00 00 00 00 00 00 00 00 00 00 00 00 00 00 00 00
 00 00 00 00 00 00 00 00 00 00 00 28 F5 FF 00 A1 2A 35 C4 84 81 83 FF 00 00 00 00 49 45 4E 44 AE
-42 60 82 00
+42 60 82 04
 EndData
 $EndBitmap
 $Bitmap
 Pos 2250 6000
-Scale 1.500000
+Scale 1,500000
 Data
 89 50 4E 47 0D 0A 1A 0A 00 00 00 0D 49 48 44 52 00 00 02 91 00 00 02 8E 08 02 00 00 00 71 C9 D5
@@
 9F DF D1 D1 31 D6 A5 40 90 E1 4D 94 96 C0 77 F7 E1 9C E9 BB 40 B5 84 6A 00 41 90 F1 06 B5 8D 23
 08 82 20 C8 04 83 62 36 82 20 08 82 4C 0C 38 D4 12 88 20 08 82 20 E3 1C 1A 1D 89 20 08 82 20 08
-82 20 08 82 20 23 ED FF 01 11 4E 07 64 6B 3C CF 2D 00 00 00 00 49 45 4E 44 AE 42 60 82 A5
+82 20 08 82 20 23 ED FF 01 11 4E 07 64 6B 3C CF 2D 00 00 00 00 49 45 4E 44 AE 42 60 82 00
 EndData
 $EndBitmap
@@
 $Bitmap
 Pos 5300 7250
-Scale 0.800000
+Scale 0,000000
 Data
 89 50 4E 47 0D 0A 1A 0A 00 00 00 0D 49 48 44 52 00 00 04 20 00 00 01 13 08 02 00 00 00 68 58 E0
@@
 L R R?
 U 1 1 558476E6
-P 7300 1550
-F 0 "R?" V 7380 1550 40  0000 C CNN
-F 1 "1M" V 7307 1551 40  0000 C CNN
-F 2 "" V 7230 1550 30  0000 C CNN
-F 3 "" H 7300 1550 30  0000 C CNN
-	1    7300 1550
+P 7700 1300
+F 0 "R?" V 7780 1300 40  0000 C CNN
+F 1 "5M" V 7707 1301 40  0000 C CNN
+F 2 "" V 7630 1300 30  0000 C CNN
+F 3 "" H 7700 1300 30  0000 C CNN
+	1    7700 1300
 	-1   0    0    1
 $EndComp
@@
 L GND #PWR05
 U 1 1 5584794D
-P 7300 1200
-F 0 "#PWR05" H 7300 1200 30  0001 C CNN
-F 1 "GND" H 7300 1130 30  0001 C CNN
-F 2 "" H 7300 1200 60  0000 C CNN
-F 3 "" H 7300 1200 60  0000 C CNN
-	1    7300 1200
+P 7700 950
+F 0 "#PWR05" H 7700 950 30  0001 C CNN
+F 1 "GND" H 7700 880 30  0001 C CNN
+F 2 "" H 7700 950 60  0000 C CNN
+F 3 "" H 7700 950 60  0000 C CNN
+	1    7700 950
 	-1   0    0    1
 $EndComp
@@
 P 6800 6250
 F 0 "R?" V 6880 6250 50  0000 C CNN
-F 1 "SHUNT" V 6800 6250 50  0000 C CNN
+F 1 "SHUNT 10K" V 6800 6250 50  0000 C CNN
 F 2 "" H 6800 6250 60  0000 C CNN
 F 3 "" H 6800 6250 60  0000 C CNN
@@
 P 6600 5650
 F 0 "R?" V 6680 5650 40  0000 C CNN
-F 1 "100" V 6607 5651 40  0000 C CNN
+F 1 "1K" V 6607 5651 40  0000 C CNN
 F 2 "" V 6530 5650 30  0000 C CNN
 F 3 "" H 6600 5650 30  0000 C CNN
@@
 P 7000 5650
 F 0 "R?" V 7080 5650 40  0000 C CNN
-F 1 "100" V 7007 5651 40  0000 C CNN
+F 1 "1K" V 7007 5651 40  0000 C CNN
 F 2 "" V 6930 5650 30  0000 C CNN
 F 3 "" H 7000 5650 30  0000 C CNN
@@
 Text Notes 4900 5800 2    30   Italic 0
 Should be high value\n
-Text Label 5900 3700 2    50   Italic 0
+Text Label 5800 3600 2    50   Italic 0
 VC10X
 $Comp
@@
 L C C?
 U 1 1 55BD1C55
-P 6950 1800
-F 0 "C?" H 6950 1900 40  0000 L CNN
-F 1 "C" H 6956 1715 40  0000 L CNN
-F 2 "" H 6988 1650 30  0000 C CNN
-F 3 "" H 6950 1800 60  0000 C CNN
-	1    6950 1800
-	-1   0    0    1
+P 7050 1300
+F 0 "C?" H 7050 1400 40  0000 L CNN
+F 1 "4,7" H 7056 1215 40  0000 L CNN
+F 2 "" H 7088 1150 30  0000 C CNN
+F 3 "" H 7050 1300 60  0000 C CNN
+	1    7050 1300
+	1    0    0    -1
 $EndComp
 $Comp
 L GND #PWR013
 U 1 1 55BD1E3F
-P 6950 2100
-F 0 "#PWR013" H 6950 2100 30  0001 C CNN
-F 1 "GND" H 6950 2030 30  0001 C CNN
-F 2 "" H 6950 2100 60  0000 C CNN
-F 3 "" H 6950 2100 60  0000 C CNN
-	1    6950 2100
-	1    0    0    -1
+P 7050 1000
+F 0 "#PWR013" H 7050 1000 30  0001 C CNN
+F 1 "GND" H 7050 930 30  0001 C CNN
+F 2 "" H 7050 1000 60  0000 C CNN
+F 3 "" H 7050 1000 60  0000 C CNN
+	1    7050 1000
+	-1   0    0    1
 $EndComp
 Text GLabel 4350 1000 0    60   Input ~ 0
@@
 P 5100 2200
 F 0 "C?" V 4950 2150 40  0000 L CNN
-F 1 "4.7u" V 5250 2150 40  0000 L CNN
+F 1 "12u" V 5250 2150 40  0000 L CNN
 F 2 "" H 5138 2050 30  0000 C CNN
 F 3 "" H 5100 2200 60  0000 C CNN
@@
 P 5000 5800
 F 0 "C?" H 5000 5900 40  0000 L CNN
-F 1 "Cf" H 5006 5715 40  0000 L CNN
+F 1 "Cf 40u" H 5006 5715 40  0000 L CNN
 F 2 "" H 5038 5650 30  0000 C CNN
 F 3 "" H 5000 5800 60  0000 C CNN
@@
 P 5000 6200
 F 0 "C?" H 5000 6300 40  0000 L CNN
-F 1 "Cf" H 5006 6115 40  0000 L CNN
+F 1 "Cf 40u" H 5006 6115 40  0000 L CNN
 F 2 "" H 5038 6050 30  0000 C CNN
 F 3 "" H 5000 6200 60  0000 C CNN
@@
 P 5000 6600
 F 0 "C?" H 5000 6700 40  0000 L CNN
-F 1 "Cf" H 5006 6515 40  0000 L CNN
+F 1 "Cf 40u" H 5006 6515 40  0000 L CNN
 F 2 "" H 5038 6450 30  0000 C CNN
 F 3 "" H 5000 6600 60  0000 C CNN
@@
 P 6150 1850
 F 0 "C?" H 6150 1950 40  0000 L CNN
-F 1 "C" H 6156 1765 40  0000 L CNN
+F 1 "10u" H 6156 1765 40  0000 L CNN
 F 2 "" H 6188 1700 30  0000 C CNN
 F 3 "" H 6150 1850 60  0000 C CNN
@@
 Text Notes 8600 5200 0    24   ~ 0
 Schottky diode for avoding high current on pin(We go to 50A+ so..)
-Text Notes 6050 2250 0    60   ~ 0
+Text Notes 5900 2250 0    60   ~ 0
 This is a ground so
 $Comp
@@
 	1    0    0    -1
 $EndComp
+Text Label 9850 1600 0    59   ~ 0
+VC10X
+Text Notes 6000 6100 0    20   ~ 0
+We are going to use 30 cell this is 15 so it's a half here it's a reason for this wierd BATT labels
+Text Notes 9150 5500 0    0    ~ 0
+And overvoltage. They value must be very close to max batt voltage
+Text Notes 8500 5700 0    28   ~ 0
+And overvoltage. value must be very close to max batt voltage.
+Text Notes 6200 5750 0    28   ~ 0
+Maybe to high value VSS and SRP will have to much  voltage diff.\n
+Text Notes 800  1450 0    59   ~ 0
+Be caerfull with VSS and other pins beacuse we must maintaine \na specific max voltage diff  between pins.\n
+Text Notes 6900 2350 0    28   ~ 0
+DSG CHG circuit TODO
+Text Notes 5600 2000 0    28   ~ 0
+VSS basicly\n
 Wire Wire Line
 	6450 2500 6450 2900
@@
 	6100 3400 6100 3700
 Wire Wire Line
-	5900 3700 6950 3700
-Wire Wire Line
-	7300 1300 7300 1200
+	7700 1050 7700 950
 Wire Wire Line
 	5300 2800 6950 2800
@@
 	7000 5150 7000 5400
 Wire Wire Line
-	6600 5400 6600 5300
-Wire Wire Line
-	6650 4700 6650 5300
-Wire Wire Line
 	7000 5300 7400 5300
 Connection ~ 7000 5300
@@
 	6650 3100 6950 3100
 Wire Wire Line
-	6650 1600 6950 1600
-Wire Wire Line
-	6950 2000 6950 2100
-Wire Wire Line
 	4350 1000 4600 1000
 Wire Wire Line
@@
 	6950 3300 6850 3300
 Wire Wire Line
-	6850 3300 6850 3600
+	6850 3300 6850 4400
 Wire Wire Line
 	6850 3600 6950 3600
@@
 	6500 4500 6500 4200
 Wire Wire Line
-	6650 4700 7500 4700
-Wire Wire Line
 	9550 1600 9550 1700
 Wire Wire Line
@@
 Wire Wire Line
 	6800 4100 6950 4100
-Wire Wire Line
-	6950 3900 6800 3900
 Connection ~ 6800 3900
 Wire Wire Line
-	7300 1800 7700 1800
-Wire Wire Line
 	8650 5300 8650 5200
 Wire Wire Line
@@
 	9300 5700 9300 3200
 Connection ~ 9300 3200
-Text Label 9850 1600 0    59   ~ 0
-VC10X
 Connection ~ 9550 1600
 Wire Wire Line
@@
 	9400 1200 9400 2600
 Connection ~ 9400 2600
-Text Notes 6000 6100 0    20   ~ 0
-We are going to use 30 cell this is 15 so it's a half here it's a reason for this wierd BATT labels
+Wire Wire Line
+	7700 1800 7700 1550
+Wire Wire Line
+	7050 1000 7050 1100
+Wire Wire Line
+	6650 1600 7050 1600
+Wire Wire Line
+	7050 1600 7050 1500
+Wire Wire Line
+	5800 3700 5800 3600
+Connection ~ 5800 3700
+Wire Wire Line
+	5500 3700 6950 3700
+Wire Wire Line
+	5100 3700 5100 3900
+Wire Wire Line
+	5100 3900 6950 3900
+$Comp
+L C C?
+U 1 1 55C2CE23
+P 5300 3700
+F 0 "C?" H 5300 3800 40  0000 L CNN
+F 1 "10u" H 5306 3615 40  0000 L CNN
+F 2 "" H 5338 3550 30  0000 C CNN
+F 3 "" H 5300 3700 60  0000 C CNN
+	1    5300 3700
+	0    -1   -1   0
+$EndComp
+Wire Wire Line
+	7500 5050 6600 5050
+Wire Wire Line
+	6600 5050 6600 5400
+Wire Wire Line
+	7500 5050 7500 4700
+Connection ~ 6850 3600
+$Comp
+L C C?
+U 1 1 55C32FBA
+P 6850 4600
+F 0 "C?" H 6850 4700 40  0000 L CNN
+F 1 "10u" H 6856 4515 40  0000 L CNN
+F 2 "" H 6888 4450 30  0000 C CNN
+F 3 "" H 6850 4600 60  0000 C CNN
+	1    6850 4600
+	1    0    0    -1
+$EndComp
+Wire Wire Line
+	6850 4800 6700 4800
+Wire Wire Line
+	6700 4800 6700 3200
+Connection ~ 6700 3200
 $EndSCHEMATC

Commit message: Fix schematic so its more readable (I think so)
Connections:
- net A: now also C?.1; no longer C?.2
- net at U?.11 (NC), U?.12 (NC), U?.14 (CAP2): now also C?.2; no longer C?.1
Other:
- note added: "This should have only low side preasumably\nI dont need current twice"
- moved on the sheet: C?, R?
