File: design/BQ7_low.sch (KiCad schematic (older format))
At the start: 41 parts

Commit message: Renew pdf set some vaules add links and more comments
Parts:
- C?: value 4.7u -> 12u
- C?: value C -> 4,7
- C? (x3): value Cf -> Cf 40u
- R?: value 1M -> 5M
- R?: value SHUNT -> SHUNT 10K
- R? (x2): value 100 -> 1K
Connections:
- net at C?.1, C?.2, R?.1: now also U?.42 (SRP)
Other:
- moved on the sheet: C?, R?
Changed lines of the file:
@@
 $Descr A4 11693 8268
 encoding utf-8
-Sheet 3 68
+Sheet 69 101
 Title "BQ76940"
 Date ""
@@
 $Bitmap
 Pos 2300 3300
-Scale 1.000000
+Scale 1,000000
 Data
 89 50 4E 47 0D 0A 1A 0A 00 00 00 0D 49 48 44 52 00 00 04 1B 00 00 02 70 08 02 00 00 00 47 C3 FE
@@
 00 00 00 00 00 00 00 00 00 00 00 00 00 00 00 00 00 00 00 00 00 00 00 00 00 00 00 00 00 00 00 00
 00 00 00 00 00 00 00 00 00 00 00 28 F5 FF 00 A1 2A 35 C4 84 81 83 FF 00 00 00 00 49 45 4E 44 AE
-42 60 82 00
+42 60 82 04
 EndData
 $EndBitmap
 $Bitmap
 Pos 2250 6000
-Scale 1.500000
+Scale 1,500000
 Data
 89 50 4E 47 0D 0A 1A 0A 00 00 00 0D 49 48 44 52 00 00 02 91 00 00 02 8E 08 02 00 00 00 71 C9 D5
@@
 9F DF D1 D1 31 D6 A5 40 90 E1 4D 94 96 C0 77 F7 E1 9C E9 BB 40 B5 84 6A 00 41 90 F1 06 B5 8D 23
 08 82 20 C8 04 83 62 36 82 20 08 82 4C 0C 38 D4 12 88 20 08 82 20 E3 1C 1A 1D 89 20 08 82 20 08
-82 20 08 82 20 23 ED FF 01 11 4E 07 64 6B 3C CF 2D 00 00 00 00 49 45 4E 44 AE 42 60 82 15
+82 20 08 82 20 23 ED FF 01 11 4E 07 64 6B 3C CF 2D 00 00 00 00 49 45 4E 44 AE 42 60 82 00
 EndData
 $EndBitmap
@@
 $Bitmap
 Pos 5300 7250
-Scale 0.800000
+Scale 0,000000
 Data
 89 50 4E 47 0D 0A 1A 0A 00 00 00 0D 49 48 44 52 00 00 04 20 00 00 01 13 08 02 00 00 00 68 58 E0
@@
 L R R?
 U 1 1 558476E6
-P 7300 1550
-F 0 "R?" V 7380 1550 40  0000 C CNN
-F 1 "1M" V 7307 1551 40  0000 C CNN
-F 2 "" V 7230 1550 30  0000 C CNN
-F 3 "" H 7300 1550 30  0000 C CNN
-	1    7300 1550
+P 7700 1300
+F 0 "R?" V 7780 1300 40  0000 C CNN
+F 1 "5M" V 7707 1301 40  0000 C CNN
+F 2 "" V 7630 1300 30  0000 C CNN
+F 3 "" H 7700 1300 30  0000 C CNN
+	1    7700 1300
 	-1   0    0    1
 $EndComp
@@
 L GND #PWR05
 U 1 1 5584794D
-P 7300 1200
-F 0 "#PWR05" H 7300 1200 30  0001 C CNN
-F 1 "GND" H 7300 1130 30  0001 C CNN
-F 2 "" H 7300 1200 60  0000 C CNN
-F 3 "" H 7300 1200 60  0000 C CNN
-	1    7300 1200
+P 7700 950
+F 0 "#PWR05" H 7700 950 30  0001 C CNN
+F 1 "GND" H 7700 880 30  0001 C CNN
+F 2 "" H 7700 950 60  0000 C CNN
+F 3 "" H 7700 950 60  0000 C CNN
+	1    7700 950
 	-1   0    0    1
 $EndComp
@@
 P 6800 6250
 F 0 "R?" V 6880 6250 50  0000 C CNN
-F 1 "SHUNT" V 6800 6250 50  0000 C CNN
+F 1 "SHUNT 10K" V 6800 6250 50  0000 C CNN
 F 2 "" H 6800 6250 60  0000 C CNN
 F 3 "" H 6800 6250 60  0000 C CNN
@@
 P 6600 5650
 F 0 "R?" V 6680 5650 40  0000 C CNN
-F 1 "100" V 6607 5651 40  0000 C CNN
+F 1 "1K" V 6607 5651 40  0000 C CNN
 F 2 "" V 6530 5650 30  0000 C CNN
 F 3 "" H 6600 5650 30  0000 C CNN
@@
 P 7000 5650
 F 0 "R?" V 7080 5650 40  0000 C CNN
-F 1 "100" V 7007 5651 40  0000 C CNN
+F 1 "1K" V 7007 5651 40  0000 C CNN
 F 2 "" V 6930 5650 30  0000 C CNN
 F 3 "" H 7000 5650 30  0000 C CNN
@@
 L C C?
 U 1 1 55BD1C55
-P 6950 1800
-F 0 "C?" H 6950 1900 40  0000 L CNN
-F 1 "C" H 6956 1715 40  0000 L CNN
-F 2 "" H 6988 1650 30  0000 C CNN
-F 3 "" H 6950 1800 60  0000 C CNN
-	1    6950 1800
-	-1   0    0    1
+P 7050 1300
+F 0 "C?" H 7050 1400 40  0000 L CNN
+F 1 "4,7" H 7056 1215 40  0000 L CNN
+F 2 "" H 7088 1150 30  0000 C CNN
+F 3 "" H 7050 1300 60  0000 C CNN
+	1    7050 1300
+	1    0    0    -1
 $EndComp
 $Comp
 L GND #PWR013
 U 1 1 55BD1E3F
-P 6950 2100
-F 0 "#PWR013" H 6950 2100 30  0001 C CNN
-F 1 "GND" H 6950 2030 30  0001 C CNN
-F 2 "" H 6950 2100 60  0000 C CNN
-F 3 "" H 6950 2100 60  0000 C CNN
-	1    6950 2100
-	1    0    0    -1
+P 7050 1000
+F 0 "#PWR013" H 7050 1000 30  0001 C CNN
+F 1 "GND" H 7050 930 30  0001 C CNN
+F 2 "" H 7050 1000 60  0000 C CNN
+F 3 "" H 7050 1000 60  0000 C CNN
+	1    7050 1000
+	-1   0    0    1
 $EndComp
 Text GLabel 4350 1000 0    60   Input ~ 0
@@
 P 5100 2200
 F 0 "C?" V 4950 2150 40  0000 L CNN
-F 1 "4.7u" V 5250 2150 40  0000 L CNN
+F 1 "12u" V 5250 2150 40  0000 L CNN
 F 2 "" H 5138 2050 30  0000 C CNN
 F 3 "" H 5100 2200 60  0000 C CNN
@@
 P 5000 5800
 F 0 "C?" H 5000 5900 40  0000 L CNN
-F 1 "Cf" H 5006 5715 40  0000 L CNN
+F 1 "Cf 40u" H 5006 5715 40  0000 L CNN
 F 2 "" H 5038 5650 30  0000 C CNN
 F 3 "" H 5000 5800 60  0000 C CNN
@@
 P 5000 6200
 F 0 "C?" H 5000 6300 40  0000 L CNN
-F 1 "Cf" H 5006 6115 40  0000 L CNN
+F 1 "Cf 40u" H 5006 6115 40  0000 L CNN
 F 2 "" H 5038 6050 30  0000 C CNN
 F 3 "" H 5000 6200 60  0000 C CNN
@@
 P 5000 6600
 F 0 "C?" H 5000 6700 40  0000 L CNN
-F 1 "Cf" H 5006 6515 40  0000 L CNN
+F 1 "Cf 40u" H 5006 6515 40  0000 L CNN
 F 2 "" H 5038 6450 30  0000 C CNN
 F 3 "" H 5000 6600 60  0000 C CNN
@@
 Text Notes 8600 5200 0    24   ~ 0
 Schottky diode for avoding high current on pin(We go to 50A+ so..)
-Text Notes 6050 2250 0    60   ~ 0
+Text Notes 5900 2250 0    60   ~ 0
 This is a ground so
 $Comp
@@
 	5900 3700 6950 3700
 Wire Wire Line
-	7300 1300 7300 1200
+	7700 1050 7700 950
 Wire Wire Line
 	5300 2800 6950 2800
@@
 	7000 5150 7000 5400
 Wire Wire Line
-	6600 5400 6600 5300
-Wire Wire Line
-	6650 4700 6650 5300
+	6600 4700 6600 5400
 Wire Wire Line
 	7000 5300 7400 5300
@@
 	6650 3100 6950 3100
 Wire Wire Line
-	6650 1600 6950 1600
-Wire Wire Line
-	6950 2000 6950 2100
-Wire Wire Line
 	4350 1000 4600 1000
 Wire Wire Line
@@
 	6500 4500 6500 4200
 Wire Wire Line
-	6650 4700 7500 4700
+	6600 4700 7500 4700
 Wire Wire Line
 	9550 1600 9550 1700
@@
 Connection ~ 6800 3900
 Wire Wire Line
-	7300 1800 7700 1800
-Wire Wire Line
 	8650 5300 8650 5200
 Wire Wire Line
@@
 Text Notes 6000 6100 0    20   ~ 0
 We are going to use 30 cell this is 15 so it's a half here it's a reason for this wierd BATT labels
+Wire Wire Line
+	7700 1800 7700 1550
+Wire Wire Line
+	7050 1000 7050 1100
+Wire Wire Line
+	6650 1600 7050 1600
+Wire Wire Line
+	7050 1600 7050 1500
 $EndSCHEMATC
