File: design/DCDC.sch (KiCad schematic (older format))
At the start: 0 parts

Commit message: Fix some mistakes and some explanations
Other:
- note added: "Short\nThis could be main DC/DC converter from batterys to motors\n20kW \nBut about 10A-30A for charing would be satisfing"
Changed lines of the file:
@@
 Text Notes 5600 650  0    60   ~ 0
 Data pins
+Text Notes 1400 2350 0    60   ~ 0
+Short\nThis could be main DC/DC converter from batterys to motors\n20kW \nBut about 10A-30A for charing would be satisfing
 $EndSCHEMATC
