File: design/MCU.sch (KiCad schematic (older format))
At the start: 0 parts

Commit message: Renew pdf set some vaules add links and more comments
Other:
- note added: "Pick any MCU you whant and make schematic or him and strat codeing"
Changed lines of the file:
@@
 $Descr A4 11693 8268
 encoding utf-8
-Sheet 2 68
+Sheet 2 101
 Title ""
 Date ""
@@
 Comment4 ""
 $EndDescr
+Text Notes 2900 1600 0    59   ~ 0
+Pick any MCU you whant and make schematic or him and strat codeing
 $EndSCHEMATC
