File: design/BQ/BQ.sch (KiCad schematic (older format))
At the start: 41 parts

Commit message: Add a new BQ and start routing board for (reason for separation for easier routing) but in the end I souldnt do this becasue of netlist but its ok because of symlink
Parts:
- removed C? (x2): Cf 40u, symbol C-RESCUE-BMS
- removed D? (x2): DIODE, symbol DIODE
- removed D? (x2): DIODESCH, symbol DIODESCH
- removed R? (x3): 50k, symbol R-RESCUE-BMS
- added C7, C8: 1u, Capacitors_SMD:C_0805, symbol C-RESCUE-BMS
- added Cf1, Cf2: 40u, Capacitors_SMD:C_1825, symbol C-RESCUE-BMS
- added D18, D19, D5: DIODE, Diodes_SMD:Diode-DO-214AB, symbol DIODE
- added D2, D3: ZENER, Diodes_SMD:SOD-123, symbol ZENER-RESCUE-BMS
- added K1: XLR3, Wire_Pads:SolderWirePad_2x_2mmDrill, symbol XLR3
- C10, C11, C6, C9: renamed from C?; footprint (none) -> Capacitors_SMD:C_0805
- C4: renamed from C?; value 12u -> 4.7; footprint (none) -> Capacitors_SMD:C_0805
- C5: renamed from C?; value C -> 1u; footprint (none) -> Capacitors_SMD:C_0805
- Cf3: renamed from C?; value Cf 40u -> 40u; footprint (none) -> Capacitors_SMD:C_1825; Name (none) -> Cf
- D1: renamed from D?; footprint (none) -> Diodes_SMD:Diode-DO-214AB
- D10, D11, D12, D13, D14, D15, D16, D17, D6, D7, D8, D9: renamed from D?; footprint (none) -> Diodes_SMD:SOD-123
- D4: renamed from D?; value DIODE -> 100V; footprint (none) -> Diodes_SMD:Diode-DO-214AB
- Q1: renamed from Q?; value MOSFET_N -> BST82,215; footprint (none) -> Transistors_SMD:sc70
- R1: renamed from R?; value Rdrain -> 200; footprint (none) -> Resistors_SMD:R_0805; Name (none) -> Rdrain
- R2: renamed from R?; value Rgate -> 100k; footprint (none) -> Resistors_SMD:R_0805; Name (none) -> Rgate
- R3: renamed from R?; value Rf 1M -> 1K; footprint (none) -> Resistors_SMD:R_0805; Name (none) -> Rf
- R4: renamed from R?; value Rd -> 100K; footprint (none) -> Resistors_SMD:R_0805
- R5, R8: renamed from R?; value 1K -> 100; footprint (none) -> Resistors_SMD:R_0805
- R6: renamed from R?; value Rsrc -> 100; footprint (none) -> Resistors_SMD:R_0805
- R7: renamed from R?; value SHUNT 10K -> SHUNT 0.001; footprint (none) -> Resistors_SMD:R_0805
- R9: renamed from R?; value 5M -> 300K; footprint (none) -> Resistors_SMD:R_0805
- U1: renamed from U?; footprint MODULE -> ab2_tssop:AB2_TSSOP44_0p50P
Connections:
- net labels added: ALERT, CHG, DSG
- wire segments 137 -> 160
Other:
- note added: "0,8 value of Schotcky"
- note added: "5,2"
- note added: "And overvoltage. They value must be very close to max batt voltage"
- note added: "And overvoltage. value must be very close to max batt voltage."
- note added: "Be caerfull with VSS and other pins beacuse we must maintaine \na specific max voltage diff between pins.\n"
- note added: "DSG CHG circuit TODO"
- note added: "For transient current"
- note added: "Gate value\n"
- note added: "In general we dont need this diodes but I would like to have them"
- note added: "Max BAT-VSS = 36V/25V\nso R must be quite high \n1K\n"
- note added: "Maybe best to be same as Rin"
- note added: "Maybe voltage and current is \nvery small so rewire this R if need"
- note added: "Reverse diode incorporated in FET"
- note added: "This pin also should be isolated"
- note added: "This should go to i2c ISO circuit"
- note added: "This should have only low side preasumably\nI dont need current twice"
- note added: "VSS basicly\n"
- note added: "Vgeth=10V\nVgs=20V(Schocht 15V)\nVds=70V\nId(const)>3A(This is to much but...)\nVregsrc=36-25V(MAX)"
- note added: "We dont whant to much voltage drop here\nVd=(60V/Ruk)*R\nRuk=R+Rdevice\nIregsrc=120uA (MAX)\n \n"
- note removed: "Max BAT-VSS = 36V/25V\nso R must be quite high \n1M"

Commit message: Add datasheets
Parts:
- K1: footprint Wire_Pads:SolderWirePad_2x_2mmDrill -> JSTcon:b2b-ph-kl
- renumbered C4 to C1, C5 to C2, C6 to C3, C7 to C4, C8 to C5, C9 to C6, C10 to C7, C11 to C8
Changed lines of the file:
@@
 00 00 00 00 00 00 00 00 00 00 00 00 00 00 00 00 00 00 00 00 00 00 00 00 00 00 00 00 00 00 00 00
 00 00 00 00 00 00 00 00 00 00 00 28 F5 FF 00 A1 2A 35 C4 84 81 83 FF 00 00 00 00 49 45 4E 44 AE
-42 60 82 11
+42 60 82 3B
 EndData
 $EndBitmap
@@
 +BATT_out
 $Comp
-L C-RESCUE-BMS C9
+L C-RESCUE-BMS C6
 U 1 1 55BCB234
 P 6800 5300
-F 0 "C9" V 6950 5250 40  0000 L CNN
+F 0 "C6" V 6950 5250 40  0000 L CNN
 F 1 "0.1u" V 6650 5250 40  0000 L CNN
 F 2 "Capacitors_SMD:C_0805" H 6838 5150 30  0001 C CNN
@@
 $EndComp
 $Comp
-L C-RESCUE-BMS C6
+L C-RESCUE-BMS C3
 U 1 1 55BCC331
 P 6250 5500
-F 0 "C6" H 6250 5600 40  0000 L CNN
+F 0 "C3" H 6250 5600 40  0000 L CNN
 F 1 "0.1u" H 6256 5415 40  0000 L CNN
 F 2 "Capacitors_SMD:C_0805" H 6288 5350 30  0001 C CNN
@@
 $EndComp
 $Comp
-L C-RESCUE-BMS C11
+L C-RESCUE-BMS C8
 U 1 1 55BCC398
 P 7400 5500
-F 0 "C11" H 7400 5600 40  0000 L CNN
+F 0 "C8" H 7400 5600 40  0000 L CNN
 F 1 "0.1u" H 7406 5415 40  0000 L CNN
 F 2 "Capacitors_SMD:C_0805" H 7438 5350 30  0001 C CNN
@@
 VC10X
 $Comp
-L C-RESCUE-BMS C10
+L C-RESCUE-BMS C7
 U 1 1 55BD1C55
 P 7050 1300
-F 0 "C10" H 7050 1400 40  0000 L CNN
+F 0 "C7" H 7050 1400 40  0000 L CNN
 F 1 "4,7" H 7056 1215 40  0000 L CNN
 F 2 "Capacitors_SMD:C_0805" H 7088 1150 30  0001 C CNN
@@
 +BATT
 $Comp
-L C-RESCUE-BMS C4
+L C-RESCUE-BMS C1
 U 1 1 55BCD3D7
 P 5700 3100
-F 0 "C4" V 5600 3050 40  0000 L CNN
+F 0 "C1" V 5600 3050 40  0000 L CNN
 F 1 "4.7" V 5850 3050 40  0000 L CNN
 F 2 "Capacitors_SMD:C_0805" H 5738 2950 30  0001 C CNN
@@
 Capactior between termistors
 $Comp
-L C-RESCUE-BMS C5
+L C-RESCUE-BMS C2
 U 1 1 55BDCF5F
 P 5850 2700
-F 0 "C5" H 5850 2800 40  0000 L CNN
+F 0 "C2" H 5850 2800 40  0000 L CNN
 F 1 "1u" H 5856 2615 40  0000 L CNN
 F 2 "Capacitors_SMD:C_0805" H 5888 2550 30  0001 C CNN
@@
 VSS basicly\n
 $Comp
-L C-RESCUE-BMS C8
+L C-RESCUE-BMS C5
 U 1 1 55C2CE23
 P 6500 3900
-F 0 "C8" H 6500 4000 40  0000 L CNN
+F 0 "C5" H 6500 4000 40  0000 L CNN
 F 1 "1u" H 6506 3815 40  0000 L CNN
 F 2 "Capacitors_SMD:C_0805" H 6538 3750 30  0001 C CNN
@@
 $EndComp
 $Comp
-L C-RESCUE-BMS C7
+L C-RESCUE-BMS C4
 U 1 1 55C32FBA
 P 6450 3400
-F 0 "C7" H 6450 3500 40  0000 L CNN
+F 0 "C4" H 6450 3500 40  0000 L CNN
 F 1 "1u" H 6456 3315 40  0000 L CNN
 F 2 "Capacitors_SMD:C_0805" H 6488 3250 30  0001 C CNN
@@
 F 0 "K1" H 10650 1100 60  0000 C CNN
 F 1 "XLR3" H 10700 600 60  0000 C CNN
-F 2 "Wire_Pads:SolderWirePad_2x_2mmDrill" H 10500 850 60  0001 C CNN
+F 2 "JSTcon:b2b-ph-kl" H 10500 850 60  0001 C CNN
 F 3 "" H 10500 850 60  0000 C CNN
 	1    10500 850
