File: design/BQ/Batt.sch (KiCad schematic (older format))
At the start: 1 part

Commit message: Add a new BQ and start routing board for (reason for separation for easier routing) but in the end I souldnt do this becasue of netlist but its ok because of symlink
Parts:
- BT6: renamed from BT?; footprint (none) -> Connect:PINHEAD1-2
Changed lines of the file:
@@
 EESchema Schematic File Version 2
-LIBS:BMS-rescue
-LIBS:iso5500
-LIBS:crf_1
-LIBS:BQ76940
+LIBS:BQ-rescue
 LIBS:power
 LIBS:device
@@
 LIBS:contrib
 LIBS:valves
-LIBS:BMS-cache
+LIBS:BQ-cache
 EELAYER 25 0
 EELAYER END
 $Descr A4 11693 8268
 encoding utf-8
-Sheet 100 101
+Sheet 100 33
 Title ""
 Date ""
@@
 AR Path="/55C14E4B/3A5B5476/3A539FA4/55BD50FF/55BBA6DA" Ref="BT?"  Part="1"
 AR Path="/55C14E4B/3A5B5476/3A54397C/55BD50FF/55BBA6DA" Ref="BT?"  Part="1"
-F 0 "BT?" H 5500 3650 50  0000 C CNN
+AR Path="/3A5B5476/3A501D31/55BD50FF/55BBA6DA" Ref="BT?"  Part="1"
+AR Path="/3A5B5476/3A5031D0/55BD50FF/55BBA6DA" Ref="BT?"  Part="1"
+AR Path="/3A5B5476/3A507C61/55BD50FF/55BBA6DA" Ref="BT?"  Part="1"
+AR Path="/3A5B5476/3A50984C/55BD50FF/55BBA6DA" Ref="BT?"  Part="1"
+AR Path="/3A5B5476/3A509CE9/55BD50FF/55BBA6DA" Ref="BT?"  Part="1"
+AR Path="/3A5B5476/3A50D488/55BD50FF/55BBA6DA" Ref="BT6"  Part="1"
+AR Path="/3A5B5476/3A51DCAC/55BD50FF/55BBA6DA" Ref="BT7"  Part="1"
+AR Path="/3A5B5476/3A53CBC8/55BD50FF/55BBA6DA" Ref="BT?"  Part="1"
+AR Path="/3A5B5476/3A5401FD/55BD50FF/55BBA6DA" Ref="BT?"  Part="1"
+AR Path="/3A5B5476/3A54231A/55BD50FF/55BBA6DA" Ref="BT?"  Part="1"
+AR Path="/3A5B5476/3A52C799/55BD50FF/55BBA6DA" Ref="BT11"  Part="1"
+AR Path="/3A5B5476/3A5314A2/55BD50FF/55BBA6DA" Ref="BT?"  Part="1"
+AR Path="/3A5B5476/3A5364FA/55BD50FF/55BBA6DA" Ref="BT?"  Part="1"
+AR Path="/3A5B5476/3A539FA4/55BD50FF/55BBA6DA" Ref="BT?"  Part="1"
+AR Path="/3A5B5476/3A54397C/55BD50FF/55BBA6DA" Ref="BT?"  Part="1"
+AR Path="/3A5B5476/3A501D31/565A4B86/55BBA6DA" Ref="BT1"  Part="1"
+AR Path="/3A5B5476/3A5031D0/565A4B86/55BBA6DA" Ref="BT2"  Part="1"
+AR Path="/3A5B5476/3A507C61/565A4B86/55BBA6DA" Ref="BT3"  Part="1"
+AR Path="/3A5B5476/3A50984C/565A4B87/55BBA6DA" Ref="BT4"  Part="1"
+AR Path="/3A5B5476/3A509CE9/565A4B86/55BBA6DA" Ref="BT5"  Part="1"
+AR Path="/3A5B5476/3A53CBC8/565A4B86/55BBA6DA" Ref="BT8"  Part="1"
+AR Path="/3A5B5476/3A5401FD/565A4B86/55BBA6DA" Ref="BT9"  Part="1"
+AR Path="/3A5B5476/3A54231A/565A4B87/55BBA6DA" Ref="BT10"  Part="1"
+AR Path="/3A5B5476/3A5314A2/565A4B86/55BBA6DA" Ref="BT12"  Part="1"
+AR Path="/3A5B5476/3A5364FA/565A4B86/55BBA6DA" Ref="BT13"  Part="1"
+AR Path="/3A5B5476/3A539FA4/565A4B86/55BBA6DA" Ref="BT14"  Part="1"
+AR Path="/3A5B5476/3A54397C/565A4B87/55BBA6DA" Ref="BT15"  Part="1"
+F 0 "BT13" H 5500 3650 50  0000 C CNN
 F 1 "BATTERY" H 5500 3260 50  0000 C CNN
-F 2 "" H 5500 3450 60  0000 C CNN
+F 2 "Connect:PINHEAD1-2" H 5500 3450 60  0001 C CNN
 F 3 "" H 5500 3450 60  0000 C CNN
 F 4 "3.7V" H 5500 3450 60  0001 C CNN "Voltage"

Commit message: Add datasheets
Parts:
- renumbered BT6 to BT1
Changed lines of the file:
@@
 $Descr A4 11693 8268
 encoding utf-8
-Sheet 100 33
+Sheet 29 33
 Title ""
 Date ""
@@
 $EndDescr
 $Comp
-L BATTERY BT?
+L BATTERY BT1
 U 1 1 55BBA6DA
 P 5500 3450
-AR Path="/55BB8FBC/3A5B5476/3A501D31/55BD50FF/55BBA6DA" Ref="BT?"  Part="1"
-AR Path="/55BB8FBC/3A5B5476/3A5031D0/55BD50FF/55BBA6DA" Ref="BT?"  Part="1"
-AR Path="/55BB8FBC/3A5B5476/3A507C61/55BD50FF/55BBA6DA" Ref="BT?"  Part="1"
-AR Path="/55BB8FBC/3A5B5476/3A50984C/55BD50FF/55BBA6DA" Ref="BT?"  Part="1"
-AR Path="/55BB8FBC/3A5B5476/3A509CE9/55BD50FF/55BBA6DA" Ref="BT?"  Part="1"
-AR Path="/55BB8FBC/3A5B5476/3A50D488/55BD50FF/55BBA6DA" Ref="BT?"  Part="1"
-AR Path="/55BB8FBC/3A5B5476/3A51DCAC/55BD50FF/55BBA6DA" Ref="BT?"  Part="1"
-AR Path="/55BB8FBC/3A5B5476/3A53CBC8/55BD50FF/55BBA6DA" Ref="BT?"  Part="1"
-AR Path="/55BB8FBC/3A5B5476/3A5401FD/55BD50FF/55BBA6DA" Ref="BT?"  Part="1"
-AR Path="/55BB8FBC/3A5B5476/3A54231A/55BD50FF/55BBA6DA" Ref="BT?"  Part="1"
-AR Path="/55BB8FBC/3A5B5476/3A52C799/55BD50FF/55BBA6DA" Ref="BT?"  Part="1"
-AR Path="/55BB8FBC/3A5B5476/3A5314A2/55BD50FF/55BBA6DA" Ref="BT?"  Part="1"
-AR Path="/55BB8FBC/3A5B5476/3A5364FA/55BD50FF/55BBA6DA" Ref="BT?"  Part="1"
-AR Path="/55BB8FBC/3A5B5476/3A539FA4/55BD50FF/55BBA6DA" Ref="BT?"  Part="1"
-AR Path="/55BB8FBC/3A5B5476/3A54397C/55BD50FF/55BBA6DA" Ref="BT?"  Part="1"
-AR Path="/55BBA6A3/55BBA6DA" Ref="BT?"  Part="1"
-AR Path="/3A58CB36/3A501D31/55BD50FF/55BBA6DA" Ref="BT?"  Part="1"
-AR Path="/3A58CB36/3A5031D0/55BD50FF/55BBA6DA" Ref="BT?"  Part="1"
-AR Path="/3A58CB36/3A507C61/55BD50FF/55BBA6DA" Ref="BT?"  Part="1"
-AR Path="/3A58CB36/3A50984C/55BD50FF/55BBA6DA" Ref="BT?"  Part="1"
-AR Path="/3A58CB36/3A509CE9/55BD50FF/55BBA6DA" Ref="BT?"  Part="1"
-AR Path="/3A58CB36/3A50D488/55BD50FF/55BBA6DA" Ref="BT?"  Part="1"
-AR Path="/3A58CB36/3A51DCAC/55BD50FF/55BBA6DA" Ref="BT?"  Part="1"
-AR Path="/3A58CB36/3A53CBC8/55BD50FF/55BBA6DA" Ref="BT?"  Part="1"
-AR Path="/3A58CB36/3A5401FD/55BD50FF/55BBA6DA" Ref="BT?"  Part="1"
-AR Path="/3A58CB36/3A54231A/55BD50FF/55BBA6DA" Ref="BT?"  Part="1"
-AR Path="/3A58CB36/3A52C799/55BD50FF/55BBA6DA" Ref="BT?"  Part="1"
-AR Path="/3A58CB36/3A5314A2/55BD50FF/55BBA6DA" Ref="BT?"  Part="1"
-AR Path="/3A58CB36/3A5364FA/55BD50FF/55BBA6DA" Ref="BT?"  Part="1"
-AR Path="/3A58CB36/3A539FA4/55BD50FF/55BBA6DA" Ref="BT?"  Part="1"
-AR Path="/3A58CB36/3A54397C/55BD50FF/55BBA6DA" Ref="BT?"  Part="1"
-AR Path="/55C14E4B/3A5B5476/3A501D31/55BD50FF/55BBA6DA" Ref="BT?"  Part="1"
-AR Path="/55C14E4B/3A5B5476/3A5031D0/55BD50FF/55BBA6DA" Ref="BT?"  Part="1"
-AR Path="/55C14E4B/3A5B5476/3A507C61/55BD50FF/55BBA6DA" Ref="BT?"  Part="1"
-AR Path="/55C14E4B/3A5B5476/3A50984C/55BD50FF/55BBA6DA" Ref="BT?"  Part="1"
-AR Path="/55C14E4B/3A5B5476/3A509CE9/55BD50FF/55BBA6DA" Ref="BT?"  Part="1"
-AR Path="/55C14E4B/3A5B5476/3A50D488/55BD50FF/55BBA6DA" Ref="BT?"  Part="1"
-AR Path="/55C14E4B/3A5B5476/3A51DCAC/55BD50FF/55BBA6DA" Ref="BT?"  Part="1"
-AR Path="/55C14E4B/3A5B5476/3A53CBC8/55BD50FF/55BBA6DA" Ref="BT?"  Part="1"
-AR Path="/55C14E4B/3A5B5476/3A5401FD/55BD50FF/55BBA6DA" Ref="BT?"  Part="1"
-AR Path="/55C14E4B/3A5B5476/3A54231A/55BD50FF/55BBA6DA" Ref="BT?"  Part="1"
-AR Path="/55C14E4B/3A5B5476/3A52C799/55BD50FF/55BBA6DA" Ref="BT?"  Part="1"
-AR Path="/55C14E4B/3A5B5476/3A5314A2/55BD50FF/55BBA6DA" Ref="BT?"  Part="1"
-AR Path="/55C14E4B/3A5B5476/3A5364FA/55BD50FF/55BBA6DA" Ref="BT?"  Part="1"
-AR Path="/55C14E4B/3A5B5476/3A539FA4/55BD50FF/55BBA6DA" Ref="BT?"  Part="1"
-AR Path="/55C14E4B/3A5B5476/3A54397C/55BD50FF/55BBA6DA" Ref="BT?"  Part="1"
-AR Path="/3A5B5476/3A501D31/55BD50FF/55BBA6DA" Ref="BT?"  Part="1"
-AR Path="/3A5B5476/3A5031D0/55BD50FF/55BBA6DA" Ref="BT?"  Part="1"
-AR Path="/3A5B5476/3A507C61/55BD50FF/55BBA6DA" Ref="BT?"  Part="1"
-AR Path="/3A5B5476/3A50984C/55BD50FF/55BBA6DA" Ref="BT?"  Part="1"
-AR Path="/3A5B5476/3A509CE9/55BD50FF/55BBA6DA" Ref="BT?"  Part="1"
-AR Path="/3A5B5476/3A50D488/55BD50FF/55BBA6DA" Ref="BT6"  Part="1"
-AR Path="/3A5B5476/3A51DCAC/55BD50FF/55BBA6DA" Ref="BT7"  Part="1"
-AR Path="/3A5B5476/3A53CBC8/55BD50FF/55BBA6DA" Ref="BT?"  Part="1"
-AR Path="/3A5B5476/3A5401FD/55BD50FF/55BBA6DA" Ref="BT?"  Part="1"
-AR Path="/3A5B5476/3A54231A/55BD50FF/55BBA6DA" Ref="BT?"  Part="1"
-AR Path="/3A5B5476/3A52C799/55BD50FF/55BBA6DA" Ref="BT11"  Part="1"
-AR Path="/3A5B5476/3A5314A2/55BD50FF/55BBA6DA" Ref="BT?"  Part="1"
-AR Path="/3A5B5476/3A5364FA/55BD50FF/55BBA6DA" Ref="BT?"  Part="1"
-AR Path="/3A5B5476/3A539FA4/55BD50FF/55BBA6DA" Ref="BT?"  Part="1"
-AR Path="/3A5B5476/3A54397C/55BD50FF/55BBA6DA" Ref="BT?"  Part="1"
 AR Path="/3A5B5476/3A501D31/565A4B86/55BBA6DA" Ref="BT1"  Part="1"
 AR Path="/3A5B5476/3A5031D0/565A4B86/55BBA6DA" Ref="BT2"  Part="1"
@@
 AR Path="/3A5B5476/3A50984C/565A4B87/55BBA6DA" Ref="BT4"  Part="1"
 AR Path="/3A5B5476/3A509CE9/565A4B86/55BBA6DA" Ref="BT5"  Part="1"
+AR Path="/3A5B5476/3A50D488/55BD50FF/55BBA6DA" Ref="BT6"  Part="1"
+AR Path="/3A5B5476/3A51DCAC/55BD50FF/55BBA6DA" Ref="BT7"  Part="1"
 AR Path="/3A5B5476/3A53CBC8/565A4B86/55BBA6DA" Ref="BT8"  Part="1"
 AR Path="/3A5B5476/3A5401FD/565A4B86/55BBA6DA" Ref="BT9"  Part="1"
 AR Path="/3A5B5476/3A54231A/565A4B87/55BBA6DA" Ref="BT10"  Part="1"
+AR Path="/3A5B5476/3A52C799/55BD50FF/55BBA6DA" Ref="BT11"  Part="1"
 AR Path="/3A5B5476/3A5314A2/565A4B86/55BBA6DA" Ref="BT12"  Part="1"
 AR Path="/3A5B5476/3A5364FA/565A4B86/55BBA6DA" Ref="BT13"  Part="1"
 AR Path="/3A5B5476/3A539FA4/565A4B86/55BBA6DA" Ref="BT14"  Part="1"
 AR Path="/3A5B5476/3A54397C/565A4B87/55BBA6DA" Ref="BT15"  Part="1"
-F 0 "BT13" H 5500 3650 50  0000 C CNN
+F 0 "BT3" H 5500 3650 50  0000 C CNN
 F 1 "BATTERY" H 5500 3260 50  0000 C CNN
 F 2 "Connect:PINHEAD1-2" H 5500 3450 60  0001 C CNN
