File: design/BQ/Batt_ball.sch (KiCad schematic (older format))
At the start: 6 parts, among them Q2 MOSFET_N

Commit message: Add datasheets
Parts:
- renumbered C15 to C12
Changed lines of the file:
@@
 $Descr A4 11693 8268
 encoding utf-8
-Sheet 4 33
+Sheet 8 33
 Title ""
 Date ""
@@
 Comment4 ""
 $EndDescr
-$Sheet
-S 4950 3700 1050 600
-U 565A4B86
-F0 "Battery cell" 60
-F1 "Batt.sch" 60
-F2 "-B" I R 6000 4000 60
-F3 "+B" I L 4950 4000 60
-$EndSheet
 Text Notes 1250 1100 0    60   ~ 0
 This is just mesurment and balancing circuit
@@
 AR Path="/3A5B5476/3A5364FA/565A4B88" Ref="R54"  Part="1"
 AR Path="/3A5B5476/3A539FA4/565A4B88" Ref="R57"  Part="1"
-F 0 "R51" V 4980 2850 40  0000 C CNN
+F 0 "R22" V 4980 2850 40  0000 C CNN
 F 1 "50" V 4907 2851 40  0000 C CNN
 F 2 "Resistors_SMD:R_0805" V 4830 2850 30  0001 C CNN
@@
 AR Path="/3A5B5476/3A5364FA/565A9525" Ref="D32"  Part="1"
 AR Path="/3A5B5476/3A539FA4/565A9525" Ref="D33"  Part="1"
-F 0 "D31" H 5900 2500 50  0000 C CNN
+F 0 "D22" H 5900 2500 50  0000 C CNN
 F 1 "5,6" H 5900 2300 40  0000 C CNN
 F 2 "Diodes_SMD:SOD-123" H 5900 2400 60  0001 C CNN
@@
 AR Path="/3A5B5476/3A5364FA/565A9528" Ref="R56"  Part="1"
 AR Path="/3A5B5476/3A539FA4/565A9528" Ref="R59"  Part="1"
-F 0 "R53" V 6480 1950 40  0000 C CNN
+F 0 "R24" V 6480 1950 40  0000 C CNN
 F 1 "1K" V 6407 1951 40  0000 C CNN
 F 2 "Resistors_SMD:R_0805" V 6330 1950 30  0001 C CNN
@@
 $EndComp
 $Comp
-L C-RESCUE-BMS C15
+L C-RESCUE-BMS C12
 U 1 1 565A9529
 P 5100 1650
-AR Path="/3A5B5476/3A501D31/565A9529" Ref="C15"  Part="1"
-AR Path="/3A5B5476/3A5031D0/565A9529" Ref="C16"  Part="1"
-AR Path="/3A5B5476/3A507C61/565A9529" Ref="C17"  Part="1"
-AR Path="/3A5B5476/3A509CE9/565A9529" Ref="C19"  Part="1"
-AR Path="/3A5B5476/3A53CBC8/565A9529" Ref="C22"  Part="1"
-AR Path="/3A5B5476/3A5401FD/565A9529" Ref="C23"  Part="1"
-AR Path="/3A5B5476/3A5314A2/565A9529" Ref="C26"  Part="1"
-AR Path="/3A5B5476/3A5364FA/565A9529" Ref="C27"  Part="1"
-AR Path="/3A5B5476/3A539FA4/565A9529" Ref="C28"  Part="1"
-F 0 "C26" V 5250 1600 40  0000 L CNN
+AR Path="/3A5B5476/3A501D31/565A9529" Ref="C12"  Part="1"
+AR Path="/3A5B5476/3A5031D0/565A9529" Ref="C13"  Part="1"
+AR Path="/3A5B5476/3A507C61/565A9529" Ref="C14"  Part="1"
+AR Path="/3A5B5476/3A509CE9/565A9529" Ref="C16"  Part="1"
+AR Path="/3A5B5476/3A53CBC8/565A9529" Ref="C19"  Part="1"
+AR Path="/3A5B5476/3A5401FD/565A9529" Ref="C20"  Part="1"
+AR Path="/3A5B5476/3A5314A2/565A9529" Ref="C23"  Part="1"
+AR Path="/3A5B5476/3A5364FA/565A9529" Ref="C24"  Part="1"
+AR Path="/3A5B5476/3A539FA4/565A9529" Ref="C25"  Part="1"
+F 0 "C14" V 5250 1600 40  0000 L CNN
 F 1 "10u" V 4950 1600 40  0000 L CNN
 F 2 "Capacitors_SMD:C_0805" H 5138 1500 30  0001 C CNN
@@
 	4500 4000 4950 4000
 Wire Wire Line
-	5150 2850 5200 2850
+	5100 2850 5200 2850
 Connection ~ 6400 2400
 Wire Wire Line
@@
 AR Path="/3A5B5476/3A5364FA/565A952B" Ref="R55"  Part="1"
 AR Path="/3A5B5476/3A539FA4/565A952B" Ref="R58"  Part="1"
-F 0 "R52" V 5480 1950 40  0000 C CNN
+F 0 "R23" V 5480 1950 40  0000 C CNN
 F 1 "10K" V 5407 1951 40  0000 C CNN
 F 2 "Resistors_SMD:R_0805" V 5330 1950 30  0001 C CNN
@@
 AR Path="/3A5B5476/3A5364FA/565A36F5" Ref="Q14"  Part="1"
 AR Path="/3A5B5476/3A539FA4/565A36F5" Ref="Q15"  Part="1"
-F 0 "Q13" H 5410 2920 60  0000 R CNN
+F 0 "Q4" H 5410 2920 60  0000 R CNN
 F 1 "MOSFET_N" H 5410 2600 60  0000 R CNN
 F 2 "CRF1:DFB1006-4" H 5400 2750 60  0001 C CNN
@@
 	0    1    1    0
 $EndComp
+Connection ~ 5150 2850
+$Sheet
+S 4950 3700 1050 600
+U 565A4B86
+F0 "Battery cell" 60
+F1 "Batt.sch" 60
+F2 "-B" I R 6000 4000 60
+F3 "+B" I L 4950 4000 60
+$EndSheet
 $EndSCHEMATC
