File: design/BQ/Batt_ball_cap.sch (KiCad schematic (older format))
At the start: 6 parts

Commit message: Add a new BQ and start routing board for (reason for separation for easier routing) but in the end I souldnt do this becasue of netlist but its ok because of symlink
Parts:
- removed D?: 5,6V, symbol ZENER-RESCUE-BMS
- removed R?: 1K, symbol R-RESCUE-BMS
- removed R?: 10K, symbol R-RESCUE-BMS
- added D25: 5,6V, Diodes_SMD:SOD-123, symbol ZENER-RESCUE-BMS
- added R33: 10K, Resistors_SMD:R_0805, symbol R-RESCUE-BMS
- added R34: 1K, Resistors_SMD:R_0805, symbol R-RESCUE-BMS
- C13: renamed from C?; footprint (none) -> Capacitors_SMD:C_0805
- Q7: renamed from Q?; footprint (none) -> CRF1:DFB1006-4
- R32: renamed from R?; footprint (none) -> Resistors_SMD:R_0805
Changed lines of the file:
@@
 EESchema Schematic File Version 2
-LIBS:BMS-rescue
-LIBS:iso5500
-LIBS:crf_1
-LIBS:BQ76940
+LIBS:BQ-rescue
 LIBS:power
 LIBS:device
@@
 LIBS:contrib
 LIBS:valves
-LIBS:BMS-cache
+LIBS:BQ-cache
 EELAYER 25 0
 EELAYER END
 $Descr A4 11693 8268
 encoding utf-8
-Sheet 26 101
+Sheet 26 33
 Title ""
 Date ""
@@
 AR Path="/55C14E4B/3A5B5476/3A51DCAC/55BD57AA" Ref="Q?"  Part="1"
 AR Path="/55C14E4B/3A5B5476/3A52C799/55BD57AA" Ref="Q?"  Part="1"
-F 0 "Q?" V 5200 2700 60  0000 R CNN
+AR Path="/3A5B5476/3A50D488/55BD57AA" Ref="Q7"  Part="1"
+AR Path="/3A5B5476/3A51DCAC/55BD57AA" Ref="Q8"  Part="1"
+AR Path="/3A5B5476/3A52C799/55BD57AA" Ref="Q12"  Part="1"
+F 0 "Q12" V 5200 2700 60  0000 R CNN
 F 1 "DMN2300UFB4-7B" V 5700 3150 60  0000 R CNN
-F 2 "" H 5400 2750 60  0000 C CNN
+F 2 "CRF1:DFB1006-4" H 5400 2750 60  0001 C CNN
 F 3 "" H 5400 2750 60  0000 C CNN
 	1    5400 2750
@@
 AR Path="/55C14E4B/3A5B5476/3A52C799/55BD5928" Ref="R?"  Part="1"
 AR Path="/55BD5928" Ref="R?"  Part="1"
-F 0 "R?" V 4980 2850 40  0000 C CNN
+AR Path="/3A5B5476/3A50D488/55BD5928" Ref="R32"  Part="1"
+AR Path="/3A5B5476/3A51DCAC/55BD5928" Ref="R35"  Part="1"
+AR Path="/3A5B5476/3A52C799/55BD5928" Ref="R48"  Part="1"
+F 0 "R48" V 4980 2850 40  0000 C CNN
 F 1 "50" V 4907 2851 40  0000 C CNN
-F 2 "" V 4830 2850 30  0000 C CNN
+F 2 "Resistors_SMD:R_0805" V 4830 2850 30  0001 C CNN
 F 3 "" H 4900 2850 30  0000 C CNN
 F 4 "Rbal" V 4900 2850 60  0001 C CNN "Name"
@@
 $Comp
 L ZENER-RESCUE-BMS D?
-U 1 1 55BD5ABC
+U 1 1 565A4B8A
 P 5900 2400
-AR Path="/55BB8FBC/3A50D488/55BD5ABC" Ref="D?"  Part="1"
-AR Path="/55BB8FBC/3A51DCAC/55BD5ABC" Ref="D?"  Part="1"
-AR Path="/55BB8FBC/55BDFAF2/55BD5ABC" Ref="D?"  Part="1"
-AR Path="/55BB8FBC/3A5B5476/3A50D488/55BD5ABC" Ref="D?"  Part="1"
-AR Path="/55BB8FBC/3A5B5476/3A51DCAC/55BD5ABC" Ref="D?"  Part="1"
-AR Path="/55BB8FBC/3A5B5476/3A52C799/55BD5ABC" Ref="D?"  Part="1"
-AR Path="/3A58CB36/3A50D488/55BD5ABC" Ref="D?"  Part="1"
-AR Path="/3A58CB36/3A51DCAC/55BD5ABC" Ref="D?"  Part="1"
-AR Path="/3A58CB36/3A52C799/55BD5ABC" Ref="D?"  Part="1"
-AR Path="/55C14E4B/3A5B5476/3A50D488/55BD5ABC" Ref="D?"  Part="1"
-AR Path="/55C14E4B/3A5B5476/3A51DCAC/55BD5ABC" Ref="D?"  Part="1"
-AR Path="/55C14E4B/3A5B5476/3A52C799/55BD5ABC" Ref="D?"  Part="1"
-F 0 "D?" H 5900 2500 50  0000 C CNN
+AR Path="/55BB8FBC/3A50D488/565A4B8A" Ref="D?"  Part="1"
+AR Path="/55BB8FBC/3A51DCAC/565A4B8A" Ref="D?"  Part="1"
+AR Path="/55BB8FBC/55BDFAF2/565A4B8A" Ref="D?"  Part="1"
+AR Path="/55BB8FBC/3A5B5476/3A50D488/565A4B8A" Ref="D?"  Part="1"
+AR Path="/55BB8FBC/3A5B5476/3A51DCAC/565A4B8A" Ref="D?"  Part="1"
+AR Path="/55BB8FBC/3A5B5476/3A52C799/565A4B8A" Ref="D?"  Part="1"
+AR Path="/3A58CB36/3A50D488/565A4B8A" Ref="D?"  Part="1"
+AR Path="/3A58CB36/3A51DCAC/565A4B8A" Ref="D?"  Part="1"
+AR Path="/3A58CB36/3A52C799/565A4B8A" Ref="D?"  Part="1"
+AR Path="/55C14E4B/3A5B5476/3A50D488/565A4B8A" Ref="D?"  Part="1"
+AR Path="/55C14E4B/3A5B5476/3A51DCAC/565A4B8A" Ref="D?"  Part="1"
+AR Path="/55C14E4B/3A5B5476/3A52C799/565A4B8A" Ref="D?"  Part="1"
+AR Path="/3A5B5476/3A50D488/565A4B8A" Ref="D25"  Part="1"
+AR Path="/3A5B5476/3A51DCAC/565A4B8A" Ref="D26"  Part="1"
+AR Path="/3A5B5476/3A52C799/565A4B8A" Ref="D30"  Part="1"
+F 0 "D30" H 5900 2500 50  0000 C CNN
 F 1 "5,6V" H 5900 2300 40  0000 C CNN
-F 2 "" H 5900 2400 60  0000 C CNN
+F 2 "Diodes_SMD:SOD-123" H 5900 2400 60  0001 C CNN
 F 3 "" H 5900 2400 60  0000 C CNN
 	1    5900 2400
@@
 $Comp
 L R-RESCUE-BMS R?
-U 1 1 55BD5B30
+U 1 1 565A4B8B
 P 6400 1950
-AR Path="/55BB8FBC/3A50D488/55BD5B30" Ref="R?"  Part="1"
-AR Path="/55BB8FBC/3A51DCAC/55BD5B30" Ref="R?"  Part="1"
-AR Path="/55BB8FBC/55BDFAF2/55BD5B30" Ref="R?"  Part="1"
-AR Path="/55BB8FBC/3A5B5476/3A50D488/55BD5B30" Ref="R?"  Part="1"
-AR Path="/55BB8FBC/3A5B5476/3A51DCAC/55BD5B30" Ref="R?"  Part="1"
-AR Path="/55BB8FBC/3A5B5476/3A52C799/55BD5B30" Ref="R?"  Part="1"
-AR Path="/3A58CB36/3A50D488/55BD5B30" Ref="R?"  Part="1"
-AR Path="/3A58CB36/3A51DCAC/55BD5B30" Ref="R?"  Part="1"
-AR Path="/3A58CB36/3A52C799/55BD5B30" Ref="R?"  Part="1"
-AR Path="/55C14E4B/3A5B5476/3A50D488/55BD5B30" Ref="R?"  Part="1"
-AR Path="/55C14E4B/3A5B5476/3A51DCAC/55BD5B30" Ref="R?"  Part="1"
-AR Path="/55C14E4B/3A5B5476/3A52C799/55BD5B30" Ref="R?"  Part="1"
-AR Path="/55BD5B30" Ref="R?"  Part="1"
-F 0 "R?" V 6480 1950 40  0000 C CNN
+AR Path="/55BB8FBC/3A50D488/565A4B8B" Ref="R?"  Part="1"
+AR Path="/55BB8FBC/3A51DCAC/565A4B8B" Ref="R?"  Part="1"
+AR Path="/55BB8FBC/55BDFAF2/565A4B8B" Ref="R?"  Part="1"
+AR Path="/55BB8FBC/3A5B5476/3A50D488/565A4B8B" Ref="R?"  Part="1"
+AR Path="/55BB8FBC/3A5B5476/3A51DCAC/565A4B8B" Ref="R?"  Part="1"
+AR Path="/55BB8FBC/3A5B5476/3A52C799/565A4B8B" Ref="R?"  Part="1"
+AR Path="/3A58CB36/3A50D488/565A4B8B" Ref="R?"  Part="1"
+AR Path="/3A58CB36/3A51DCAC/565A4B8B" Ref="R?"  Part="1"
+AR Path="/3A58CB36/3A52C799/565A4B8B" Ref="R?"  Part="1"
+AR Path="/55C14E4B/3A5B5476/3A50D488/565A4B8B" Ref="R?"  Part="1"
+AR Path="/55C14E4B/3A5B5476/3A51DCAC/565A4B8B" Ref="R?"  Part="1"
+AR Path="/55C14E4B/3A5B5476/3A52C799/565A4B8B" Ref="R?"  Part="1"
+AR Path="/565A4B8B" Ref="R?"  Part="1"
+AR Path="/3A5B5476/3A50D488/565A4B8B" Ref="R34"  Part="1"
+AR Path="/3A5B5476/3A51DCAC/565A4B8B" Ref="R37"  Part="1"
+AR Path="/3A5B5476/3A52C799/565A4B8B" Ref="R50"  Part="1"
+F 0 "R50" V 6480 1950 40  0000 C CNN
 F 1 "1K" V 6407 1951 40  0000 C CNN
-F 2 "" V 6330 1950 30  0000 C CNN
+F 2 "Resistors_SMD:R_0805" V 6330 1950 30  0001 C CNN
 F 3 "" H 6400 1950 30  0000 C CNN
 	1    6400 1950
@@
 AR Path="/55C14E4B/3A5B5476/3A52C799/55BD5F3E" Ref="C?"  Part="1"
 AR Path="/55BD5F3E" Ref="C?"  Part="1"
-F 0 "C?" V 5250 1600 40  0000 L CNN
+AR Path="/3A5B5476/3A50D488/55BD5F3E" Ref="C13"  Part="1"
+AR Path="/3A5B5476/3A51DCAC/55BD5F3E" Ref="C14"  Part="1"
+AR Path="/3A5B5476/3A52C799/55BD5F3E" Ref="C20"  Part="1"
+F 0 "C20" V 5250 1600 40  0000 L CNN
 F 1 "10u" V 4950 1600 40  0000 L CNN
-F 2 "" H 5138 1500 30  0000 C CNN
+F 2 "Capacitors_SMD:C_0805" H 5138 1500 30  0001 C CNN
 F 3 "" H 5100 1650 60  0000 C CNN
 F 4 "Cc" V 5100 1650 60  0001 C CNN "Name"
@@
 $Comp
 L R-RESCUE-BMS R?
-U 1 1 55BD60D7
+U 1 1 565A4B8D
 P 5400 1950
-AR Path="/55BB8FBC/3A50D488/55BD60D7" Ref="R?"  Part="1"
-AR Path="/55BB8FBC/3A51DCAC/55BD60D7" Ref="R?"  Part="1"
-AR Path="/55BB8FBC/55BDFAF2/55BD60D7" Ref="R?"  Part="1"
-AR Path="/55BB8FBC/3A5B5476/3A50D488/55BD60D7" Ref="R?"  Part="1"
-AR Path="/55BB8FBC/3A5B5476/3A51DCAC/55BD60D7" Ref="R?"  Part="1"
-AR Path="/55BB8FBC/3A5B5476/3A52C799/55BD60D7" Ref="R?"  Part="1"
-AR Path="/3A58CB36/3A50D488/55BD60D7" Ref="R?"  Part="1"
-AR Path="/3A58CB36/3A51DCAC/55BD60D7" Ref="R?"  Part="1"
-AR Path="/3A58CB36/3A52C799/55BD60D7" Ref="R?"  Part="1"
-AR Path="/55C14E4B/3A5B5476/3A50D488/55BD60D7" Ref="R?"  Part="1"
-AR Path="/55C14E4B/3A5B5476/3A51DCAC/55BD60D7" Ref="R?"  Part="1"
-AR Path="/55C14E4B/3A5B5476/3A52C799/55BD60D7" Ref="R?"  Part="1"
-AR Path="/55BD60D7" Ref="R?"  Part="1"
-F 0 "R?" V 5480 1950 40  0000 C CNN
+AR Path="/55BB8FBC/3A50D488/565A4B8D" Ref="R?"  Part="1"
+AR Path="/55BB8FBC/3A51DCAC/565A4B8D" Ref="R?"  Part="1"
+AR Path="/55BB8FBC/55BDFAF2/565A4B8D" Ref="R?"  Part="1"
+AR Path="/55BB8FBC/3A5B5476/3A50D488/565A4B8D" Ref="R?"  Part="1"
+AR Path="/55BB8FBC/3A5B5476/3A51DCAC/565A4B8D" Ref="R?"  Part="1"
+AR Path="/55BB8FBC/3A5B5476/3A52C799/565A4B8D" Ref="R?"  Part="1"
+AR Path="/3A58CB36/3A50D488/565A4B8D" Ref="R?"  Part="1"
+AR Path="/3A58CB36/3A51DCAC/565A4B8D" Ref="R?"  Part="1"
+AR Path="/3A58CB36/3A52C799/565A4B8D" Ref="R?"  Part="1"
+AR Path="/55C14E4B/3A5B5476/3A50D488/565A4B8D" Ref="R?"  Part="1"
+AR Path="/55C14E4B/3A5B5476/3A51DCAC/565A4B8D" Ref="R?"  Part="1"
+AR Path="/55C14E4B/3A5B5476/3A52C799/565A4B8D" Ref="R?"  Part="1"
+AR Path="/565A4B8D" Ref="R?"  Part="1"
+AR Path="/3A5B5476/3A50D488/565A4B8D" Ref="R33"  Part="1"
+AR Path="/3A5B5476/3A51DCAC/565A4B8D" Ref="R36"  Part="1"
+AR Path="/3A5B5476/3A52C799/565A4B8D" Ref="R49"  Part="1"
+F 0 "R49" V 5480 1950 40  0000 C CNN
 F 1 "10K" V 5407 1951 40  0000 C CNN
-F 2 "" V 5330 1950 30  0000 C CNN
+F 2 "Resistors_SMD:R_0805" V 5330 1950 30  0001 C CNN
 F 3 "" H 5400 1950 30  0000 C CNN
 	1    5400 1950

Commit message: Add datasheets
Parts:
- renumbered C13 to C17
Changed lines of the file:
@@
 $Descr A4 11693 8268
 encoding utf-8
-Sheet 26 33
+Sheet 24 33
 Title ""
 Date ""
@@
 This is just mesurment and balancing circuit
 $Comp
-L MOS_N Q?
+L MOS_N Q7
 U 1 1 55BD57AA
 P 5400 2750
-AR Path="/55BB8FBC/3A50D488/55BD57AA" Ref="Q?"  Part="1"
-AR Path="/55BB8FBC/3A51DCAC/55BD57AA" Ref="Q?"  Part="1"
-AR Path="/55BB8FBC/55BDFAF2/55BD57AA" Ref="Q?"  Part="1"
-AR Path="/55BB8FBC/3A5B5476/3A50D488/55BD57AA" Ref="Q?"  Part="1"
-AR Path="/55BB8FBC/3A5B5476/3A51DCAC/55BD57AA" Ref="Q?"  Part="1"
-AR Path="/55BB8FBC/3A5B5476/3A52C799/55BD57AA" Ref="Q?"  Part="1"
-AR Path="/3A58CB36/3A50D488/55BD57AA" Ref="Q?"  Part="1"
-AR Path="/3A58CB36/3A51DCAC/55BD57AA" Ref="Q?"  Part="1"
-AR Path="/3A58CB36/3A52C799/55BD57AA" Ref="Q?"  Part="1"
-AR Path="/55C14E4B/3A5B5476/3A50D488/55BD57AA" Ref="Q?"  Part="1"
-AR Path="/55C14E4B/3A5B5476/3A51DCAC/55BD57AA" Ref="Q?"  Part="1"
-AR Path="/55C14E4B/3A5B5476/3A52C799/55BD57AA" Ref="Q?"  Part="1"
 AR Path="/3A5B5476/3A50D488/55BD57AA" Ref="Q7"  Part="1"
 AR Path="/3A5B5476/3A51DCAC/55BD57AA" Ref="Q8"  Part="1"
 AR Path="/3A5B5476/3A52C799/55BD57AA" Ref="Q12"  Part="1"
-F 0 "Q12" V 5200 2700 60  0000 R CNN
+F 0 "Q7" V 5200 2700 60  0000 R CNN
 F 1 "DMN2300UFB4-7B" V 5700 3150 60  0000 R CNN
 F 2 "CRF1:DFB1006-4" H 5400 2750 60  0001 C CNN
@@
 $EndComp
 $Comp
-L R-RESCUE-BMS R?
+L R-RESCUE-BMS R32
 U 1 1 55BD5928
 P 4900 2850
-AR Path="/55BB8FBC/3A50D488/55BD5928" Ref="R?"  Part="1"
-AR Path="/55BB8FBC/3A51DCAC/55BD5928" Ref="R?"  Part="1"
-AR Path="/55BB8FBC/55BDFAF2/55BD5928" Ref="R?"  Part="1"
-AR Path="/55BB8FBC/3A5B5476/3A50D488/55BD5928" Ref="R?"  Part="1"
-AR Path="/55BB8FBC/3A5B5476/3A51DCAC/55BD5928" Ref="R?"  Part="1"
-AR Path="/55BB8FBC/3A5B5476/3A52C799/55BD5928" Ref="R?"  Part="1"
-AR Path="/3A58CB36/3A50D488/55BD5928" Ref="R?"  Part="1"
-AR Path="/3A58CB36/3A51DCAC/55BD5928" Ref="R?"  Part="1"
-AR Path="/3A58CB36/3A52C799/55BD5928" Ref="R?"  Part="1"
-AR Path="/55C14E4B/3A5B5476/3A50D488/55BD5928" Ref="R?"  Part="1"
-AR Path="/55C14E4B/3A5B5476/3A51DCAC/55BD5928" Ref="R?"  Part="1"
-AR Path="/55C14E4B/3A5B5476/3A52C799/55BD5928" Ref="R?"  Part="1"
-AR Path="/55BD5928" Ref="R?"  Part="1"
 AR Path="/3A5B5476/3A50D488/55BD5928" Ref="R32"  Part="1"
 AR Path="/3A5B5476/3A51DCAC/55BD5928" Ref="R35"  Part="1"
 AR Path="/3A5B5476/3A52C799/55BD5928" Ref="R48"  Part="1"
-F 0 "R48" V 4980 2850 40  0000 C CNN
+F 0 "R32" V 4980 2850 40  0000 C CNN
 F 1 "50" V 4907 2851 40  0000 C CNN
 F 2 "Resistors_SMD:R_0805" V 4830 2850 30  0001 C CNN
@@
 $EndComp
 $Comp
-L ZENER-RESCUE-BMS D?
+L ZENER-RESCUE-BMS D25
 U 1 1 565A4B8A
 P 5900 2400
-AR Path="/55BB8FBC/3A50D488/565A4B8A" Ref="D?"  Part="1"
-AR Path="/55BB8FBC/3A51DCAC/565A4B8A" Ref="D?"  Part="1"
-AR Path="/55BB8FBC/55BDFAF2/565A4B8A" Ref="D?"  Part="1"
-AR Path="/55BB8FBC/3A5B5476/3A50D488/565A4B8A" Ref="D?"  Part="1"
-AR Path="/55BB8FBC/3A5B5476/3A51DCAC/565A4B8A" Ref="D?"  Part="1"
-AR Path="/55BB8FBC/3A5B5476/3A52C799/565A4B8A" Ref="D?"  Part="1"
-AR Path="/3A58CB36/3A50D488/565A4B8A" Ref="D?"  Part="1"
-AR Path="/3A58CB36/3A51DCAC/565A4B8A" Ref="D?"  Part="1"
-AR Path="/3A58CB36/3A52C799/565A4B8A" Ref="D?"  Part="1"
-AR Path="/55C14E4B/3A5B5476/3A50D488/565A4B8A" Ref="D?"  Part="1"
-AR Path="/55C14E4B/3A5B5476/3A51DCAC/565A4B8A" Ref="D?"  Part="1"
-AR Path="/55C14E4B/3A5B5476/3A52C799/565A4B8A" Ref="D?"  Part="1"
 AR Path="/3A5B5476/3A50D488/565A4B8A" Ref="D25"  Part="1"
 AR Path="/3A5B5476/3A51DCAC/565A4B8A" Ref="D26"  Part="1"
 AR Path="/3A5B5476/3A52C799/565A4B8A" Ref="D30"  Part="1"
-F 0 "D30" H 5900 2500 50  0000 C CNN
+F 0 "D25" H 5900 2500 50  0000 C CNN
 F 1 "5,6V" H 5900 2300 40  0000 C CNN
 F 2 "Diodes_SMD:SOD-123" H 5900 2400 60  0001 C CNN
@@
 $EndComp
 $Comp
-L R-RESCUE-BMS R?
+L R-RESCUE-BMS R34
 U 1 1 565A4B8B
 P 6400 1950
-AR Path="/55BB8FBC/3A50D488/565A4B8B" Ref="R?"  Part="1"
-AR Path="/55BB8FBC/3A51DCAC/565A4B8B" Ref="R?"  Part="1"
-AR Path="/55BB8FBC/55BDFAF2/565A4B8B" Ref="R?"  Part="1"
-AR Path="/55BB8FBC/3A5B5476/3A50D488/565A4B8B" Ref="R?"  Part="1"
-AR Path="/55BB8FBC/3A5B5476/3A51DCAC/565A4B8B" Ref="R?"  Part="1"
-AR Path="/55BB8FBC/3A5B5476/3A52C799/565A4B8B" Ref="R?"  Part="1"
-AR Path="/3A58CB36/3A50D488/565A4B8B" Ref="R?"  Part="1"
-AR Path="/3A58CB36/3A51DCAC/565A4B8B" Ref="R?"  Part="1"
-AR Path="/3A58CB36/3A52C799/565A4B8B" Ref="R?"  Part="1"
-AR Path="/55C14E4B/3A5B5476/3A50D488/565A4B8B" Ref="R?"  Part="1"
-AR Path="/55C14E4B/3A5B5476/3A51DCAC/565A4B8B" Ref="R?"  Part="1"
-AR Path="/55C14E4B/3A5B5476/3A52C799/565A4B8B" Ref="R?"  Part="1"
-AR Path="/565A4B8B" Ref="R?"  Part="1"
 AR Path="/3A5B5476/3A50D488/565A4B8B" Ref="R34"  Part="1"
 AR Path="/3A5B5476/3A51DCAC/565A4B8B" Ref="R37"  Part="1"
 AR Path="/3A5B5476/3A52C799/565A4B8B" Ref="R50"  Part="1"
-F 0 "R50" V 6480 1950 40  0000 C CNN
+F 0 "R34" V 6480 1950 40  0000 C CNN
 F 1 "1K" V 6407 1951 40  0000 C CNN
 F 2 "Resistors_SMD:R_0805" V 6330 1950 30  0001 C CNN
@@
 $EndComp
 $Comp
-L C-RESCUE-BMS C?
+L C-RESCUE-BMS C17
 U 1 1 55BD5F3E
 P 5100 1650
-AR Path="/55BB8FBC/3A50D488/55BD5F3E" Ref="C?"  Part="1"
-AR Path="/55BB8FBC/3A51DCAC/55BD5F3E" Ref="C?"  Part="1"
-AR Path="/55BB8FBC/55BDFAF2/55BD5F3E" Ref="C?"  Part="1"
-AR Path="/55BB8FBC/3A5B5476/3A50D488/55BD5F3E" Ref="C?"  Part="1"
-AR Path="/55BB8FBC/3A5B5476/3A51DCAC/55BD5F3E" Ref="C?"  Part="1"
-AR Path="/55BB8FBC/3A5B5476/3A52C799/55BD5F3E" Ref="C?"  Part="1"
-AR Path="/3A58CB36/3A50D488/55BD5F3E" Ref="C?"  Part="1"
-AR Path="/3A58CB36/3A51DCAC/55BD5F3E" Ref="C?"  Part="1"
-AR Path="/3A58CB36/3A52C799/55BD5F3E" Ref="C?"  Part="1"
-AR Path="/55C14E4B/3A5B5476/3A50D488/55BD5F3E" Ref="C?"  Part="1"
-AR Path="/55C14E4B/3A5B5476/3A51DCAC/55BD5F3E" Ref="C?"  Part="1"
-AR Path="/55C14E4B/3A5B5476/3A52C799/55BD5F3E" Ref="C?"  Part="1"
-AR Path="/55BD5F3E" Ref="C?"  Part="1"
-AR Path="/3A5B5476/3A50D488/55BD5F3E" Ref="C13"  Part="1"
-AR Path="/3A5B5476/3A51DCAC/55BD5F3E" Ref="C14"  Part="1"
-AR Path="/3A5B5476/3A52C799/55BD5F3E" Ref="C20"  Part="1"
-F 0 "C20" V 5250 1600 40  0000 L CNN
+AR Path="/3A5B5476/3A50D488/55BD5F3E" Ref="C17"  Part="1"
+AR Path="/3A5B5476/3A51DCAC/55BD5F3E" Ref="C18"  Part="1"
+AR Path="/3A5B5476/3A52C799/55BD5F3E" Ref="C22"  Part="1"
+F 0 "C17" V 5250 1600 40  0000 L CNN
 F 1 "10u" V 4950 1600 40  0000 L CNN
 F 2 "Capacitors_SMD:C_0805" H 5138 1500 30  0001 C CNN
@@
 $EndComp
 $Comp
-L R-RESCUE-BMS R?
+L R-RESCUE-BMS R33
 U 1 1 565A4B8D
 P 5400 1950
-AR Path="/55BB8FBC/3A50D488/565A4B8D" Ref="R?"  Part="1"
-AR Path="/55BB8FBC/3A51DCAC/565A4B8D" Ref="R?"  Part="1"
-AR Path="/55BB8FBC/55BDFAF2/565A4B8D" Ref="R?"  Part="1"
-AR Path="/55BB8FBC/3A5B5476/3A50D488/565A4B8D" Ref="R?"  Part="1"
-AR Path="/55BB8FBC/3A5B5476/3A51DCAC/565A4B8D" Ref="R?"  Part="1"
-AR Path="/55BB8FBC/3A5B5476/3A52C799/565A4B8D" Ref="R?"  Part="1"
-AR Path="/3A58CB36/3A50D488/565A4B8D" Ref="R?"  Part="1"
-AR Path="/3A58CB36/3A51DCAC/565A4B8D" Ref="R?"  Part="1"
-AR Path="/3A58CB36/3A52C799/565A4B8D" Ref="R?"  Part="1"
-AR Path="/55C14E4B/3A5B5476/3A50D488/565A4B8D" Ref="R?"  Part="1"
-AR Path="/55C14E4B/3A5B5476/3A51DCAC/565A4B8D" Ref="R?"  Part="1"
-AR Path="/55C14E4B/3A5B5476/3A52C799/565A4B8D" Ref="R?"  Part="1"
-AR Path="/565A4B8D" Ref="R?"  Part="1"
 AR Path="/3A5B5476/3A50D488/565A4B8D" Ref="R33"  Part="1"
 AR Path="/3A5B5476/3A51DCAC/565A4B8D" Ref="R36"  Part="1"
 AR Path="/3A5B5476/3A52C799/565A4B8D" Ref="R49"  Part="1"
-F 0 "R49" V 5480 1950 40  0000 C CNN
+F 0 "R33" V 5480 1950 40  0000 C CNN
 F 1 "10K" V 5407 1951 40  0000 C CNN
 F 2 "Resistors_SMD:R_0805" V 5330 1950 30  0001 C CNN
