File: design/BQ/Batt_ball_end.sch (KiCad schematic (older format))
At the start: 7 parts

Commit message: Add a new BQ and start routing board for (reason for separation for easier routing) but in the end I souldnt do this becasue of netlist but its ok because of symlink
Parts:
- removed C?: 10u, symbol C-RESCUE-BMS
- removed R?: 50, symbol R-RESCUE-BMS
- added C12: 10u, Capacitors_SMD:C_0805, symbol C-RESCUE-BMS
- added R26: 50, Resistors_SMD:R_0805, symbol R-RESCUE-BMS
- D23: renamed from D?; footprint (none) -> Diodes_SMD:SOD-123
- Q5: renamed from Q?; footprint (none) -> CRF1:DFB1006-4
- R25, R27, R28: renamed from R?; footprint (none) -> Resistors_SMD:R_0805
Changed lines of the file:
@@
 EESchema Schematic File Version 2
-LIBS:BMS-rescue
-LIBS:iso5500
-LIBS:crf_1
-LIBS:BQ76940
+LIBS:BQ-rescue
 LIBS:power
 LIBS:device
@@
 LIBS:contrib
 LIBS:valves
-LIBS:BMS-cache
+LIBS:BQ-cache
 EELAYER 25 0
 EELAYER END
 $Descr A4 11693 8268
 encoding utf-8
-Sheet 34 101
+Sheet 34 33
 Title ""
 Date ""
@@
 $Sheet
 S 4950 3700 1050 600
-U 55BD50FF
+U 565A4B87
 F0 "Battery cell" 60
 F1 "Batt.sch" 60
@@
 $Comp
 L R-RESCUE-BMS R?
-U 1 1 55BD5928
+U 1 1 565A4B89
 P 4900 2850
-AR Path="/55BB8FBC/3A50D488/55BD5928" Ref="R?"  Part="1"
-AR Path="/55BB8FBC/3A51DCAC/55BD5928" Ref="R?"  Part="1"
-AR Path="/55BB8FBC/3A50984C/55BD5928" Ref="R?"  Part="1"
-AR Path="/55BB8FBC/3A5B5476/3A50984C/55BD5928" Ref="R?"  Part="1"
-AR Path="/55BB8FBC/3A5B5476/3A54231A/55BD5928" Ref="R?"  Part="1"
-AR Path="/55BB8FBC/3A5B5476/3A54397C/55BD5928" Ref="R?"  Part="1"
-AR Path="/3A58CB36/3A50984C/55BD5928" Ref="R?"  Part="1"
-AR Path="/3A58CB36/3A54231A/55BD5928" Ref="R?"  Part="1"
-AR Path="/3A58CB36/3A54397C/55BD5928" Ref="R?"  Part="1"
-AR Path="/55C14E4B/3A5B5476/3A50984C/55BD5928" Ref="R?"  Part="1"
-AR Path="/55C14E4B/3A5B5476/3A54231A/55BD5928" Ref="R?"  Part="1"
-AR Path="/55C14E4B/3A5B5476/3A54397C/55BD5928" Ref="R?"  Part="1"
-AR Path="/55BD5928" Ref="R?"  Part="1"
-F 0 "R?" V 4980 2850 40  0000 C CNN
+AR Path="/55BB8FBC/3A50D488/565A4B89" Ref="R?"  Part="1"
+AR Path="/55BB8FBC/3A51DCAC/565A4B89" Ref="R?"  Part="1"
+AR Path="/55BB8FBC/3A50984C/565A4B89" Ref="R?"  Part="1"
+AR Path="/55BB8FBC/3A5B5476/3A50984C/565A4B89" Ref="R?"  Part="1"
+AR Path="/55BB8FBC/3A5B5476/3A54231A/565A4B89" Ref="R?"  Part="1"
+AR Path="/55BB8FBC/3A5B5476/3A54397C/565A4B89" Ref="R?"  Part="1"
+AR Path="/3A58CB36/3A50984C/565A4B89" Ref="R?"  Part="1"
+AR Path="/3A58CB36/3A54231A/565A4B89" Ref="R?"  Part="1"
+AR Path="/3A58CB36/3A54397C/565A4B89" Ref="R?"  Part="1"
+AR Path="/55C14E4B/3A5B5476/3A50984C/565A4B89" Ref="R?"  Part="1"
+AR Path="/55C14E4B/3A5B5476/3A54231A/565A4B89" Ref="R?"  Part="1"
+AR Path="/55C14E4B/3A5B5476/3A54397C/565A4B89" Ref="R?"  Part="1"
+AR Path="/565A4B89" Ref="R?"  Part="1"
+AR Path="/3A5B5476/3A50984C/565A4B89" Ref="R26"  Part="1"
+AR Path="/3A5B5476/3A54231A/565A4B89" Ref="R45"  Part="1"
+AR Path="/3A5B5476/3A54397C/565A4B89" Ref="R61"  Part="1"
+F 0 "R26" V 4980 2850 40  0000 C CNN
 F 1 "50" V 4907 2851 40  0000 C CNN
-F 2 "" V 4830 2850 30  0000 C CNN
+F 2 "Resistors_SMD:R_0805" V 4830 2850 30  0001 C CNN
 F 3 "" H 4900 2850 30  0000 C CNN
 	1    4900 2850
@@
 AR Path="/55C14E4B/3A5B5476/3A54231A/55BD5ABC" Ref="D?"  Part="1"
 AR Path="/55C14E4B/3A5B5476/3A54397C/55BD5ABC" Ref="D?"  Part="1"
-F 0 "D?" H 5900 2500 50  0000 C CNN
+AR Path="/3A5B5476/3A50984C/55BD5ABC" Ref="D23"  Part="1"
+AR Path="/3A5B5476/3A54231A/55BD5ABC" Ref="D29"  Part="1"
+AR Path="/3A5B5476/3A54397C/55BD5ABC" Ref="D34"  Part="1"
+F 0 "D23" H 5900 2500 50  0000 C CNN
 F 1 "5,6" H 5900 2300 40  0000 C CNN
-F 2 "" H 5900 2400 60  0000 C CNN
+F 2 "Diodes_SMD:SOD-123" H 5900 2400 60  0001 C CNN
 F 3 "" H 5900 2400 60  0000 C CNN
 	1    5900 2400
@@
 AR Path="/55C14E4B/3A5B5476/3A54397C/55BD5B30" Ref="R?"  Part="1"
 AR Path="/55BD5B30" Ref="R?"  Part="1"
-F 0 "R?" V 6480 1950 40  0000 C CNN
+AR Path="/3A5B5476/3A50984C/55BD5B30" Ref="R28"  Part="1"
+AR Path="/3A5B5476/3A54231A/55BD5B30" Ref="R47"  Part="1"
+AR Path="/3A5B5476/3A54397C/55BD5B30" Ref="R63"  Part="1"
+F 0 "R28" V 6480 1950 40  0000 C CNN
 F 1 "1K" V 6407 1951 40  0000 C CNN
-F 2 "" V 6330 1950 30  0000 C CNN
+F 2 "Resistors_SMD:R_0805" V 6330 1950 30  0001 C CNN
 F 3 "" H 6400 1950 30  0000 C CNN
 F 4 "Rc" V 6400 1950 60  0001 C CNN "Name"
@@
 AR Path="/55C14E4B/3A5B5476/3A54397C/55BD5E1E" Ref="R?"  Part="1"
 AR Path="/55BD5E1E" Ref="R?"  Part="1"
-F 0 "R?" V 4580 2250 40  0000 C CNN
+AR Path="/3A5B5476/3A50984C/55BD5E1E" Ref="R25"  Part="1"
+AR Path="/3A5B5476/3A54231A/55BD5E1E" Ref="R44"  Part="1"
+AR Path="/3A5B5476/3A54397C/55BD5E1E" Ref="R60"  Part="1"
+F 0 "R25" V 4580 2250 40  0000 C CNN
 F 1 "1K" V 4507 2251 40  0000 C CNN
-F 2 "" V 4430 2250 30  0000 C CNN
+F 2 "Resistors_SMD:R_0805" V 4430 2250 30  0001 C CNN
 F 3 "" H 4500 2250 30  0000 C CNN
 	1    4500 2250
@@
 $Comp
 L C-RESCUE-BMS C?
-U 1 1 55BD5F3E
+U 1 1 565A4B8C
 P 5100 1650
-AR Path="/55BB8FBC/3A50D488/55BD5F3E" Ref="C?"  Part="1"
-AR Path="/55BB8FBC/3A51DCAC/55BD5F3E" Ref="C?"  Part="1"
-AR Path="/55BB8FBC/3A50984C/55BD5F3E" Ref="C?"  Part="1"
-AR Path="/55BB8FBC/3A5B5476/3A50984C/55BD5F3E" Ref="C?"  Part="1"
-AR Path="/55BB8FBC/3A5B5476/3A54231A/55BD5F3E" Ref="C?"  Part="1"
-AR Path="/55BB8FBC/3A5B5476/3A54397C/55BD5F3E" Ref="C?"  Part="1"
-AR Path="/3A58CB36/3A50984C/55BD5F3E" Ref="C?"  Part="1"
-AR Path="/3A58CB36/3A54231A/55BD5F3E" Ref="C?"  Part="1"
-AR Path="/3A58CB36/3A54397C/55BD5F3E" Ref="C?"  Part="1"
-AR Path="/55C14E4B/3A5B5476/3A50984C/55BD5F3E" Ref="C?"  Part="1"
-AR Path="/55C14E4B/3A5B5476/3A54231A/55BD5F3E" Ref="C?"  Part="1"
-AR Path="/55C14E4B/3A5B5476/3A54397C/55BD5F3E" Ref="C?"  Part="1"
-AR Path="/55BD5F3E" Ref="C?"  Part="1"
-F 0 "C?" V 5250 1600 40  0000 L CNN
+AR Path="/55BB8FBC/3A50D488/565A4B8C" Ref="C?"  Part="1"
+AR Path="/55BB8FBC/3A51DCAC/565A4B8C" Ref="C?"  Part="1"
+AR Path="/55BB8FBC/3A50984C/565A4B8C" Ref="C?"  Part="1"
+AR Path="/55BB8FBC/3A5B5476/3A50984C/565A4B8C" Ref="C?"  Part="1"
+AR Path="/55BB8FBC/3A5B5476/3A54231A/565A4B8C" Ref="C?"  Part="1"
+AR Path="/55BB8FBC/3A5B5476/3A54397C/565A4B8C" Ref="C?"  Part="1"
+AR Path="/3A58CB36/3A50984C/565A4B8C" Ref="C?"  Part="1"
+AR Path="/3A58CB36/3A54231A/565A4B8C" Ref="C?"  Part="1"
+AR Path="/3A58CB36/3A54397C/565A4B8C" Ref="C?"  Part="1"
+AR Path="/55C14E4B/3A5B5476/3A50984C/565A4B8C" Ref="C?"  Part="1"
+AR Path="/55C14E4B/3A5B5476/3A54231A/565A4B8C" Ref="C?"  Part="1"
+AR Path="/55C14E4B/3A5B5476/3A54397C/565A4B8C" Ref="C?"  Part="1"
+AR Path="/565A4B8C" Ref="C?"  Part="1"
+AR Path="/3A5B5476/3A50984C/565A4B8C" Ref="C12"  Part="1"
+AR Path="/3A5B5476/3A54231A/565A4B8C" Ref="C18"  Part="1"
+AR Path="/3A5B5476/3A54397C/565A4B8C" Ref="C21"  Part="1"
+F 0 "C12" V 5250 1600 40  0000 L CNN
 F 1 "10u" V 4950 1600 40  0000 L CNN
-F 2 "" H 5138 1500 30  0000 C CNN
+F 2 "Capacitors_SMD:C_0805" H 5138 1500 30  0001 C CNN
 F 3 "" H 5100 1650 60  0000 C CNN
 F 4 "Cc" V 5100 1650 60  0001 C CNN "Name"
@@
 AR Path="/55C14E4B/3A5B5476/3A54397C/55BD60D7" Ref="R?"  Part="1"
 AR Path="/55BD60D7" Ref="R?"  Part="1"
-F 0 "R?" V 5480 1950 40  0000 C CNN
+AR Path="/3A5B5476/3A50984C/55BD60D7" Ref="R27"  Part="1"
+AR Path="/3A5B5476/3A54231A/55BD60D7" Ref="R46"  Part="1"
+AR Path="/3A5B5476/3A54397C/55BD60D7" Ref="R62"  Part="1"
+F 0 "R27" V 5480 1950 40  0000 C CNN
 F 1 "10K" V 5407 1951 40  0000 C CNN
-F 2 "" V 5330 1950 30  0000 C CNN
+F 2 "Resistors_SMD:R_0805" V 5330 1950 30  0001 C CNN
 F 3 "" H 5400 1950 30  0000 C CNN
 	1    5400 1950
@@
 	4500 4000 4950 4000
 $Comp
-L MOSFET_N Q?
+L MOSFET_N Q5
 U 1 1 565A31AE
 P 5400 2750
-F 0 "Q?" H 5410 2920 60  0000 R CNN
+AR Path="/3A5B5476/3A50984C/565A31AE" Ref="Q5"  Part="1"
+AR Path="/3A5B5476/3A54231A/565A31AE" Ref="Q11"  Part="1"
+AR Path="/3A5B5476/3A54397C/565A31AE" Ref="Q16"  Part="1"
+F 0 "Q5" H 5410 2920 60  0000 R CNN
 F 1 "MOSFET_N" H 5410 2600 60  0000 R CNN
-F 2 "" H 5400 2750 60  0000 C CNN
+F 2 "CRF1:DFB1006-4" H 5400 2750 60  0001 C CNN
 F 3 "" H 5400 2750 60  0000 C CNN
 	1    5400 2750

Commit message: Add datasheets
Parts:
- renumbered C12 to C15
Changed lines of the file:
@@
 $Descr A4 11693 8268
 encoding utf-8
-Sheet 34 33
+Sheet 32 33
 Title ""
 Date ""
@@
 This is just mesurment and balancing circuit
 $Comp
-L R-RESCUE-BMS R?
+L R-RESCUE-BMS R26
 U 1 1 565A4B89
 P 4900 2850
-AR Path="/55BB8FBC/3A50D488/565A4B89" Ref="R?"  Part="1"
-AR Path="/55BB8FBC/3A51DCAC/565A4B89" Ref="R?"  Part="1"
-AR Path="/55BB8FBC/3A50984C/565A4B89" Ref="R?"  Part="1"
-AR Path="/55BB8FBC/3A5B5476/3A50984C/565A4B89" Ref="R?"  Part="1"
-AR Path="/55BB8FBC/3A5B5476/3A54231A/565A4B89" Ref="R?"  Part="1"
-AR Path="/55BB8FBC/3A5B5476/3A54397C/565A4B89" Ref="R?"  Part="1"
-AR Path="/3A58CB36/3A50984C/565A4B89" Ref="R?"  Part="1"
-AR Path="/3A58CB36/3A54231A/565A4B89" Ref="R?"  Part="1"
-AR Path="/3A58CB36/3A54397C/565A4B89" Ref="R?"  Part="1"
-AR Path="/55C14E4B/3A5B5476/3A50984C/565A4B89" Ref="R?"  Part="1"
-AR Path="/55C14E4B/3A5B5476/3A54231A/565A4B89" Ref="R?"  Part="1"
-AR Path="/55C14E4B/3A5B5476/3A54397C/565A4B89" Ref="R?"  Part="1"
-AR Path="/565A4B89" Ref="R?"  Part="1"
 AR Path="/3A5B5476/3A50984C/565A4B89" Ref="R26"  Part="1"
 AR Path="/3A5B5476/3A54231A/565A4B89" Ref="R45"  Part="1"
@@
 $EndComp
 $Comp
-L ZENER-RESCUE-BMS D?
+L ZENER-RESCUE-BMS D23
 U 1 1 55BD5ABC
 P 5900 2400
-AR Path="/55BB8FBC/3A50D488/55BD5ABC" Ref="D?"  Part="1"
-AR Path="/55BB8FBC/3A51DCAC/55BD5ABC" Ref="D?"  Part="1"
-AR Path="/55BB8FBC/3A50984C/55BD5ABC" Ref="D?"  Part="1"
-AR Path="/55BB8FBC/3A5B5476/3A50984C/55BD5ABC" Ref="D?"  Part="1"
-AR Path="/55BB8FBC/3A5B5476/3A54231A/55BD5ABC" Ref="D?"  Part="1"
-AR Path="/55BB8FBC/3A5B5476/3A54397C/55BD5ABC" Ref="D?"  Part="1"
-AR Path="/3A58CB36/3A50984C/55BD5ABC" Ref="D?"  Part="1"
-AR Path="/3A58CB36/3A54231A/55BD5ABC" Ref="D?"  Part="1"
-AR Path="/3A58CB36/3A54397C/55BD5ABC" Ref="D?"  Part="1"
-AR Path="/55C14E4B/3A5B5476/3A50984C/55BD5ABC" Ref="D?"  Part="1"
-AR Path="/55C14E4B/3A5B5476/3A54231A/55BD5ABC" Ref="D?"  Part="1"
-AR Path="/55C14E4B/3A5B5476/3A54397C/55BD5ABC" Ref="D?"  Part="1"
 AR Path="/3A5B5476/3A50984C/55BD5ABC" Ref="D23"  Part="1"
 AR Path="/3A5B5476/3A54231A/55BD5ABC" Ref="D29"  Part="1"
@@
 $EndComp
 $Comp
-L R-RESCUE-BMS R?
+L R-RESCUE-BMS R28
 U 1 1 55BD5B30
 P 6400 1950
-AR Path="/55BB8FBC/3A50D488/55BD5B30" Ref="R?"  Part="1"
-AR Path="/55BB8FBC/3A51DCAC/55BD5B30" Ref="R?"  Part="1"
-AR Path="/55BB8FBC/3A50984C/55BD5B30" Ref="R?"  Part="1"
-AR Path="/55BB8FBC/3A5B5476/3A50984C/55BD5B30" Ref="R?"  Part="1"
-AR Path="/55BB8FBC/3A5B5476/3A54231A/55BD5B30" Ref="R?"  Part="1"
-AR Path="/55BB8FBC/3A5B5476/3A54397C/55BD5B30" Ref="R?"  Part="1"
-AR Path="/3A58CB36/3A50984C/55BD5B30" Ref="R?"  Part="1"
-AR Path="/3A58CB36/3A54231A/55BD5B30" Ref="R?"  Part="1"
-AR Path="/3A58CB36/3A54397C/55BD5B30" Ref="R?"  Part="1"
-AR Path="/55C14E4B/3A5B5476/3A50984C/55BD5B30" Ref="R?"  Part="1"
-AR Path="/55C14E4B/3A5B5476/3A54231A/55BD5B30" Ref="R?"  Part="1"
-AR Path="/55C14E4B/3A5B5476/3A54397C/55BD5B30" Ref="R?"  Part="1"
-AR Path="/55BD5B30" Ref="R?"  Part="1"
 AR Path="/3A5B5476/3A50984C/55BD5B30" Ref="R28"  Part="1"
 AR Path="/3A5B5476/3A54231A/55BD5B30" Ref="R47"  Part="1"
@@
 $EndComp
 $Comp
-L R-RESCUE-BMS R?
+L R-RESCUE-BMS R25
 U 1 1 55BD5E1E
 P 4500 2250
-AR Path="/55BB8FBC/3A50D488/55BD5E1E" Ref="R?"  Part="1"
-AR Path="/55BB8FBC/3A51DCAC/55BD5E1E" Ref="R?"  Part="1"
-AR Path="/55BB8FBC/3A50984C/55BD5E1E" Ref="R?"  Part="1"
-AR Path="/55BB8FBC/3A5B5476/3A50984C/55BD5E1E" Ref="R?"  Part="1"
-AR Path="/55BB8FBC/3A5B5476/3A54231A/55BD5E1E" Ref="R?"  Part="1"
-AR Path="/55BB8FBC/3A5B5476/3A54397C/55BD5E1E" Ref="R?"  Part="1"
-AR Path="/3A58CB36/3A50984C/55BD5E1E" Ref="R?"  Part="1"
-AR Path="/3A58CB36/3A54231A/55BD5E1E" Ref="R?"  Part="1"
-AR Path="/3A58CB36/3A54397C/55BD5E1E" Ref="R?"  Part="1"
-AR Path="/55C14E4B/3A5B5476/3A50984C/55BD5E1E" Ref="R?"  Part="1"
-AR Path="/55C14E4B/3A5B5476/3A54231A/55BD5E1E" Ref="R?"  Part="1"
-AR Path="/55C14E4B/3A5B5476/3A54397C/55BD5E1E" Ref="R?"  Part="1"
-AR Path="/55BD5E1E" Ref="R?"  Part="1"
 AR Path="/3A5B5476/3A50984C/55BD5E1E" Ref="R25"  Part="1"
 AR Path="/3A5B5476/3A54231A/55BD5E1E" Ref="R44"  Part="1"
@@
 $EndComp
 $Comp
-L C-RESCUE-BMS C?
+L C-RESCUE-BMS C15
 U 1 1 565A4B8C
 P 5100 1650
-AR Path="/55BB8FBC/3A50D488/565A4B8C" Ref="C?"  Part="1"
-AR Path="/55BB8FBC/3A51DCAC/565A4B8C" Ref="C?"  Part="1"
-AR Path="/55BB8FBC/3A50984C/565A4B8C" Ref="C?"  Part="1"
-AR Path="/55BB8FBC/3A5B5476/3A50984C/565A4B8C" Ref="C?"  Part="1"
-AR Path="/55BB8FBC/3A5B5476/3A54231A/565A4B8C" Ref="C?"  Part="1"
-AR Path="/55BB8FBC/3A5B5476/3A54397C/565A4B8C" Ref="C?"  Part="1"
-AR Path="/3A58CB36/3A50984C/565A4B8C" Ref="C?"  Part="1"
-AR Path="/3A58CB36/3A54231A/565A4B8C" Ref="C?"  Part="1"
-AR Path="/3A58CB36/3A54397C/565A4B8C" Ref="C?"  Part="1"
-AR Path="/55C14E4B/3A5B5476/3A50984C/565A4B8C" Ref="C?"  Part="1"
-AR Path="/55C14E4B/3A5B5476/3A54231A/565A4B8C" Ref="C?"  Part="1"
-AR Path="/55C14E4B/3A5B5476/3A54397C/565A4B8C" Ref="C?"  Part="1"
-AR Path="/565A4B8C" Ref="C?"  Part="1"
-AR Path="/3A5B5476/3A50984C/565A4B8C" Ref="C12"  Part="1"
-AR Path="/3A5B5476/3A54231A/565A4B8C" Ref="C18"  Part="1"
-AR Path="/3A5B5476/3A54397C/565A4B8C" Ref="C21"  Part="1"
-F 0 "C12" V 5250 1600 40  0000 L CNN
+AR Path="/3A5B5476/3A50984C/565A4B8C" Ref="C15"  Part="1"
+AR Path="/3A5B5476/3A54231A/565A4B8C" Ref="C21"  Part="1"
+AR Path="/3A5B5476/3A54397C/565A4B8C" Ref="C26"  Part="1"
+F 0 "C15" V 5250 1600 40  0000 L CNN
 F 1 "10u" V 4950 1600 40  0000 L CNN
 F 2 "Capacitors_SMD:C_0805" H 5138 1500 30  0001 C CNN
@@
 $EndComp
 $Comp
-L R-RESCUE-BMS R?
+L R-RESCUE-BMS R27
 U 1 1 55BD60D7
 P 5400 1950
-AR Path="/55BB8FBC/3A50D488/55BD60D7" Ref="R?"  Part="1"
-AR Path="/55BB8FBC/3A51DCAC/55BD60D7" Ref="R?"  Part="1"
-AR Path="/55BB8FBC/3A50984C/55BD60D7" Ref="R?"  Part="1"
-AR Path="/55BB8FBC/3A5B5476/3A50984C/55BD60D7" Ref="R?"  Part="1"
-AR Path="/55BB8FBC/3A5B5476/3A54231A/55BD60D7" Ref="R?"  Part="1"
-AR Path="/55BB8FBC/3A5B5476/3A54397C/55BD60D7" Ref="R?"  Part="1"
-AR Path="/3A58CB36/3A50984C/55BD60D7" Ref="R?"  Part="1"
-AR Path="/3A58CB36/3A54231A/55BD60D7" Ref="R?"  Part="1"
-AR Path="/3A58CB36/3A54397C/55BD60D7" Ref="R?"  Part="1"
-AR Path="/55C14E4B/3A5B5476/3A50984C/55BD60D7" Ref="R?"  Part="1"
-AR Path="/55C14E4B/3A5B5476/3A54231A/55BD60D7" Ref="R?"  Part="1"
-AR Path="/55C14E4B/3A5B5476/3A54397C/55BD60D7" Ref="R?"  Part="1"
-AR Path="/55BD60D7" Ref="R?"  Part="1"
 AR Path="/3A5B5476/3A50984C/55BD60D7" Ref="R27"  Part="1"
 AR Path="/3A5B5476/3A54231A/55BD60D7" Ref="R46"  Part="1"
