File: design/BQ/Batt_pack.sch (KiCad schematic (older format))
At the start: 6 parts

Commit message: Add a new BQ and start routing board for (reason for separation for easier routing) but in the end I souldnt do this becasue of netlist but its ok because of symlink
Parts:
- Cc1: renamed from Cc?; footprint (none) -> Capacitors_SMD:C_0805
- Cc2: renamed from C?; footprint (none) -> Capacitors_SMD:C_0805
- Cc5: footprint (none) -> Capacitors_SMD:C_0805
- R: footprint (none) -> Resistors_SMD:R_0805
- R13, R14: renamed from R?; footprint (none) -> Resistors_SMD:R_0805
Changed lines of the file:
@@
 EESchema Schematic File Version 2
-LIBS:BMS-rescue
-LIBS:iso5500
-LIBS:crf_1
-LIBS:BQ76940
+LIBS:BQ-rescue
 LIBS:power
 LIBS:device
@@
 LIBS:contrib
 LIBS:valves
-LIBS:BMS-cache
+LIBS:BQ-cache
 EELAYER 25 0
 EELAYER END
 $Descr A4 11693 8268
 encoding utf-8
-Sheet 5 101
+Sheet 3 33
 Title "Battery Pack"
 Date ""
@@
 AR Path="/55C14E4B/3A5B5476/3A50FF92" Ref="R"  Part="1"
 AR Path="/3A50FF92" Ref="R"  Part="1"
-F 0 "R" V 6630 4400 40  0000 C CNN
+AR Path="/3A5B5476/3A50FF92" Ref="R15"  Part="1"
+F 0 "R15" V 6630 4400 40  0000 C CNN
 F 1 "1K" V 6557 4401 40  0000 C CNN
-F 2 "" V 6480 4400 30  0000 C CNN
+F 2 "Resistors_SMD:R_0805" V 6480 4400 30  0001 C CNN
 F 3 "" H 6550 4400 30  0000 C CNN
 	1    6550 4400
@@
 AR Path="/55C14E4B/3A5B5476/3A513D90" Ref="Cc5"  Part="1"
 AR Path="/3A513D90" Ref="Cc?"  Part="1"
-F 0 "Cc?" H 6450 4250 40  0000 L CNN
+AR Path="/3A5B5476/3A513D90" Ref="Cc3"  Part="1"
+F 0 "Cc3" H 6450 4250 40  0000 L CNN
 F 1 "1ou" H 6456 4065 40  0000 L CNN
-F 2 "" H 6488 4000 30  0000 C CNN
+F 2 "Capacitors_SMD:C_0805" H 6488 4000 30  0001 C CNN
 F 3 "" H 6450 4150 60  0000 C CNN
 	1    6450 4150
@@
 AR Path="/55C14E4B/3A5B5476/3A5210D8" Ref="R?"  Part="1"
 AR Path="/3A5210D8" Ref="R?"  Part="1"
-F 0 "R?" V 6580 6100 40  0000 C CNN
+AR Path="/3A5B5476/3A5210D8" Ref="R13"  Part="1"
+F 0 "R13" V 6580 6100 40  0000 C CNN
 F 1 "1K" V 6507 6101 40  0000 C CNN
-F 2 "" V 6430 6100 30  0000 C CNN
+F 2 "Resistors_SMD:R_0805" V 6430 6100 30  0001 C CNN
 F 3 "" H 6500 6100 30  0000 C CNN
 	1    6500 6100
@@
 AR Path="/55C14E4B/3A5B5476/3A5210DE" Ref="Cc?"  Part="1"
 AR Path="/3A5210DE" Ref="Cc?"  Part="1"
-F 0 "Cc?" H 6400 5950 40  0000 L CNN
+AR Path="/3A5B5476/3A5210DE" Ref="Cc1"  Part="1"
+F 0 "Cc1" H 6400 5950 40  0000 L CNN
 F 1 "10u" H 6406 5765 40  0000 L CNN
-F 2 "" H 6438 5700 30  0000 C CNN
+F 2 "Capacitors_SMD:C_0805" H 6438 5700 30  0001 C CNN
 F 3 "" H 6400 5850 60  0000 C CNN
 	1    6400 5850
@@
 AR Path="/55C14E4B/3A5B5476/3A53561F" Ref="R?"  Part="1"
 AR Path="/3A53561F" Ref="R?"  Part="1"
-F 0 "R?" V 6630 2700 40  0000 C CNN
+AR Path="/3A5B5476/3A53561F" Ref="R14"  Part="1"
+F 0 "R14" V 6630 2700 40  0000 C CNN
 F 1 "1K" V 6557 2701 40  0000 C CNN
-F 2 "" V 6480 2700 30  0000 C CNN
+F 2 "Resistors_SMD:R_0805" V 6480 2700 30  0001 C CNN
 F 3 "" H 6550 2700 30  0000 C CNN
 	1    6550 2700
@@
 Mess bellow. Batt_ball circuit are sharing every pin expect last and first\nSo becase they are sharing pin they are sharing a Rin so only\nlast should have it.(IN every block).
 $Comp
-L C C?
+L C Cc2
 U 1 1 565BDFD2
 P 6450 2450
-F 0 "C?" H 6475 2550 50  0000 L CNN
+F 0 "Cc2" H 6475 2550 50  0000 L CNN
 F 1 "10u" H 6475 2350 50  0000 L CNN
-F 2 "" H 6488 2300 30  0000 C CNN
+F 2 "Capacitors_SMD:C_0805" H 6488 2300 30  0001 C CNN
 F 3 "" H 6450 2450 60  0000 C CNN
 	1    6450 2450

Commit message: Add datasheets
Parts:
- renumbered Cc5 to Cc3, R to R15
Changed lines of the file:
@@
 $EndSheet
 $Comp
-L R-RESCUE-BMS R
+L R-RESCUE-BMS R15
 U 1 1 3A50FF92
 P 6550 4400
-AR Path="/55BB8FBC/3A5B5476/3A50FF92" Ref="R"  Part="1"
-AR Path="/3A58CB36/3A50FF92" Ref="R"  Part="1"
-AR Path="/55C14E4B/3A5B5476/3A50FF92" Ref="R"  Part="1"
-AR Path="/3A50FF92" Ref="R"  Part="1"
-AR Path="/3A5B5476/3A50FF92" Ref="R15"  Part="1"
 F 0 "R15" V 6630 4400 40  0000 C CNN
 F 1 "1K" V 6557 4401 40  0000 C CNN
@@
 $EndComp
 $Comp
-L C-RESCUE-BMS Cc?
+L C-RESCUE-BMS Cc3
 U 1 1 3A513D90
 P 6450 4150
-AR Path="/55BB8FBC/3A5B5476/3A513D90" Ref="Cc?"  Part="1"
-AR Path="/3A58CB36/3A513D90" Ref="Cc5"  Part="1"
-AR Path="/55C14E4B/3A5B5476/3A513D90" Ref="Cc5"  Part="1"
-AR Path="/3A513D90" Ref="Cc?"  Part="1"
-AR Path="/3A5B5476/3A513D90" Ref="Cc3"  Part="1"
 F 0 "Cc3" H 6450 4250 40  0000 L CNN
 F 1 "1ou" H 6456 4065 40  0000 L CNN
@@
 $EndComp
 $Comp
-L R-RESCUE-BMS R?
+L R-RESCUE-BMS R13
 U 1 1 3A5210D8
 P 6500 6100
-AR Path="/55BB8FBC/3A5B5476/3A5210D8" Ref="R?"  Part="1"
-AR Path="/3A58CB36/3A5210D8" Ref="R?"  Part="1"
-AR Path="/55C14E4B/3A5B5476/3A5210D8" Ref="R?"  Part="1"
-AR Path="/3A5210D8" Ref="R?"  Part="1"
-AR Path="/3A5B5476/3A5210D8" Ref="R13"  Part="1"
 F 0 "R13" V 6580 6100 40  0000 C CNN
 F 1 "1K" V 6507 6101 40  0000 C CNN
@@
 $EndComp
 $Comp
-L C-RESCUE-BMS Cc?
+L C-RESCUE-BMS Cc1
 U 1 1 3A5210DE
 P 6400 5850
-AR Path="/55BB8FBC/3A5B5476/3A5210DE" Ref="Cc?"  Part="1"
-AR Path="/3A58CB36/3A5210DE" Ref="Cc?"  Part="1"
-AR Path="/55C14E4B/3A5B5476/3A5210DE" Ref="Cc?"  Part="1"
-AR Path="/3A5210DE" Ref="Cc?"  Part="1"
-AR Path="/3A5B5476/3A5210DE" Ref="Cc1"  Part="1"
 F 0 "Cc1" H 6400 5950 40  0000 L CNN
 F 1 "10u" H 6406 5765 40  0000 L CNN
@@
 $EndSheet
 $Comp
-L R-RESCUE-BMS R?
+L R-RESCUE-BMS R14
 U 1 1 3A53561F
 P 6550 2700
-AR Path="/55BB8FBC/3A5B5476/3A53561F" Ref="R?"  Part="1"
-AR Path="/3A58CB36/3A53561F" Ref="R?"  Part="1"
-AR Path="/55C14E4B/3A5B5476/3A53561F" Ref="R?"  Part="1"
-AR Path="/3A53561F" Ref="R?"  Part="1"
-AR Path="/3A5B5476/3A53561F" Ref="R14"  Part="1"
 F 0 "R14" V 6630 2700 40  0000 C CNN
 F 1 "1K" V 6557 2701 40  0000 C CNN
