File: design/BQ/Temp.sch (KiCad schematic (older format))
At the start: 6 parts

Commit message: Add a new BQ and start routing board for (reason for separation for easier routing) but in the end I souldnt do this becasue of netlist but its ok because of symlink
Parts:
- C1, C2, C3: renamed from C?; footprint (none) -> Capacitors_SMD:C_0805
- R10, R11, R12: renamed from R?; footprint (none) -> Resistors_SMD:R_0805
Changed lines of the file:
@@
 EESchema Schematic File Version 2
-LIBS:BMS-rescue
-LIBS:iso5500
-LIBS:crf_1
-LIBS:BQ76940
+LIBS:BQ-rescue
 LIBS:power
 LIBS:device
@@
 LIBS:contrib
 LIBS:valves
-LIBS:BMS-cache
+LIBS:BQ-cache
 EELAYER 25 0
 EELAYER END
 $Descr A4 11693 8268
 encoding utf-8
-Sheet 69 101
+Sheet 69 33
 Title ""
 Date ""
@@
 AR Path="/55C14E4B/55844E2F/55845069" Ref="R?"  Part="1"
 AR Path="/55845069" Ref="R?"  Part="1"
-F 0 "R?" V 4580 2350 40  0000 C CNN
+AR Path="/55844E2F/55845069" Ref="R10"  Part="1"
+F 0 "R10" V 4580 2350 40  0000 C CNN
 F 1 "NTC 10k" V 4507 2351 40  0000 C CNN
-F 2 "" V 4430 2350 30  0000 C CNN
+F 2 "Resistors_SMD:R_0805" V 4430 2350 30  0001 C CNN
 F 3 "" H 4500 2350 30  0000 C CNN
 	1    4500 2350
@@
 AR Path="/55C14E4B/55844E2F/558451B7" Ref="R?"  Part="1"
 AR Path="/558451B7" Ref="R?"  Part="1"
-F 0 "R?" V 4580 2550 40  0000 C CNN
+AR Path="/55844E2F/558451B7" Ref="R11"  Part="1"
+F 0 "R11" V 4580 2550 40  0000 C CNN
 F 1 "NTC 10k" V 4507 2551 40  0000 C CNN
-F 2 "" V 4430 2550 30  0000 C CNN
+F 2 "Resistors_SMD:R_0805" V 4430 2550 30  0001 C CNN
 F 3 "" H 4500 2550 30  0000 C CNN
 	1    4500 2550
@@
 AR Path="/55C14E4B/55844E2F/558451FF" Ref="R?"  Part="1"
 AR Path="/558451FF" Ref="R?"  Part="1"
-F 0 "R?" V 4580 2750 40  0000 C CNN
+AR Path="/55844E2F/558451FF" Ref="R12"  Part="1"
+F 0 "R12" V 4580 2750 40  0000 C CNN
 F 1 "NTC 10k" V 4507 2751 40  0000 C CNN
-F 2 "" V 4430 2750 30  0000 C CNN
+F 2 "Resistors_SMD:R_0805" V 4430 2750 30  0001 C CNN
 F 3 "" H 4500 2750 30  0000 C CNN
 	1    4500 2750
@@
 82 20 08 82 20 08 82 20 08 82 20 08 82 20 08 82 20 08 82 20 08 82 20 08 82 20 08 82 20 08 82 20
 08 82 20 08 82 20 08 82 20 08 82 20 08 82 20 08 62 42 FE 1F B4 B0 EA B8 71 1B 11 2A 00 00 00 00
-49 45 4E 44 AE 42 60 82 21
+49 45 4E 44 AE 42 60 82 D1
 EndData
 $EndBitmap
@@
 AR Path="/55C14E4B/55844E2F/55DF2E2F" Ref="C?"  Part="1"
 AR Path="/55DF2E2F" Ref="C?"  Part="1"
-F 0 "C?" V 4350 3200 40  0000 L CNN
+AR Path="/55844E2F/55DF2E2F" Ref="C2"  Part="1"
+F 0 "C2" V 4350 3200 40  0000 L CNN
 F 1 "4.7" V 4600 3200 40  0000 L CNN
-F 2 "" H 4538 3100 30  0000 C CNN
+F 2 "Capacitors_SMD:C_0805" H 4538 3100 30  0001 C CNN
 F 3 "" H 4500 3250 60  0000 C CNN
 	1    4500 3250
@@
 AR Path="/55C14E4B/55844E2F/55DF2F28" Ref="C?"  Part="1"
 AR Path="/55DF2F28" Ref="C?"  Part="1"
-F 0 "C?" V 4400 3500 40  0000 L CNN
+AR Path="/55844E2F/55DF2F28" Ref="C3"  Part="1"
+F 0 "C3" V 4400 3500 40  0000 L CNN
 F 1 "4.7" V 4650 3500 40  0000 L CNN
-F 2 "" H 4538 3400 30  0000 C CNN
+F 2 "Capacitors_SMD:C_0805" H 4538 3400 30  0001 C CNN
 F 3 "" H 4500 3550 60  0000 C CNN
 	1    4500 3550
@@
 AR Path="/55C14E4B/55844E2F/55DF2F5C" Ref="C?"  Part="1"
 AR Path="/55DF2F5C" Ref="C?"  Part="1"
-F 0 "C?" V 4350 1850 40  0000 L CNN
+AR Path="/55844E2F/55DF2F5C" Ref="C1"  Part="1"
+F 0 "C1" V 4350 1850 40  0000 L CNN
 F 1 "4.7" V 4650 1850 40  0000 L CNN
-F 2 "" H 4538 1750 30  0000 C CNN
+F 2 "Capacitors_SMD:C_0805" H 4538 1750 30  0001 C CNN
 F 3 "" H 4500 1900 60  0000 C CNN
 	1    4500 1900

Commit message: Add datasheets
Parts:
- renumbered C2 to C10, C3 to C11, C1 to C9
Changed lines of the file:
@@
 $EndDescr
 $Comp
-L R-RESCUE-BMS R?
+L R-RESCUE-BMS R10
 U 1 1 55845069
 P 4500 2350
-AR Path="/55BB8FBC/55844E2F/55845069" Ref="R?"  Part="1"
-AR Path="/55C14E4B/55844E2F/55845069" Ref="R?"  Part="1"
-AR Path="/55845069" Ref="R?"  Part="1"
-AR Path="/55844E2F/55845069" Ref="R10"  Part="1"
 F 0 "R10" V 4580 2350 40  0000 C CNN
 F 1 "NTC 10k" V 4507 2351 40  0000 C CNN
@@
 $EndComp
 $Comp
-L R-RESCUE-BMS R?
+L R-RESCUE-BMS R11
 U 1 1 558451B7
 P 4500 2550
-AR Path="/55BB8FBC/55844E2F/558451B7" Ref="R?"  Part="1"
-AR Path="/55C14E4B/55844E2F/558451B7" Ref="R?"  Part="1"
-AR Path="/558451B7" Ref="R?"  Part="1"
-AR Path="/55844E2F/558451B7" Ref="R11"  Part="1"
 F 0 "R11" V 4580 2550 40  0000 C CNN
 F 1 "NTC 10k" V 4507 2551 40  0000 C CNN
@@
 $EndComp
 $Comp
-L R-RESCUE-BMS R?
+L R-RESCUE-BMS R12
 U 1 1 558451FF
 P 4500 2750
-AR Path="/55BB8FBC/55844E2F/558451FF" Ref="R?"  Part="1"
-AR Path="/55C14E4B/55844E2F/558451FF" Ref="R?"  Part="1"
-AR Path="/558451FF" Ref="R?"  Part="1"
-AR Path="/55844E2F/558451FF" Ref="R12"  Part="1"
 F 0 "R12" V 4580 2750 40  0000 C CNN
 F 1 "NTC 10k" V 4507 2751 40  0000 C CNN
@@
 82 20 08 82 20 08 82 20 08 82 20 08 82 20 08 82 20 08 82 20 08 82 20 08 82 20 08 82 20 08 82 20
 08 82 20 08 82 20 08 82 20 08 82 20 08 82 20 08 62 42 FE 1F B4 B0 EA B8 71 1B 11 2A 00 00 00 00
-49 45 4E 44 AE 42 60 82 D1
+49 45 4E 44 AE 42 60 82 61
 EndData
 $EndBitmap
@@
 Missing only for NTC so we can convert to Temp
 $Comp
-L C-RESCUE-BMS C?
+L C-RESCUE-BMS C10
 U 1 1 55DF2E2F
 P 4500 3250
-AR Path="/55BB8FBC/55844E2F/55DF2E2F" Ref="C?"  Part="1"
-AR Path="/55C14E4B/55844E2F/55DF2E2F" Ref="C?"  Part="1"
-AR Path="/55DF2E2F" Ref="C?"  Part="1"
-AR Path="/55844E2F/55DF2E2F" Ref="C2"  Part="1"
-F 0 "C2" V 4350 3200 40  0000 L CNN
+F 0 "C10" V 4350 3200 40  0000 L CNN
 F 1 "4.7" V 4600 3200 40  0000 L CNN
 F 2 "Capacitors_SMD:C_0805" H 4538 3100 30  0001 C CNN
@@
 $EndComp
 $Comp
-L C-RESCUE-BMS C?
+L C-RESCUE-BMS C11
 U 1 1 55DF2F28
 P 4500 3550
-AR Path="/55BB8FBC/55844E2F/55DF2F28" Ref="C?"  Part="1"
-AR Path="/55C14E4B/55844E2F/55DF2F28" Ref="C?"  Part="1"
-AR Path="/55DF2F28" Ref="C?"  Part="1"
-AR Path="/55844E2F/55DF2F28" Ref="C3"  Part="1"
-F 0 "C3" V 4400 3500 40  0000 L CNN
+F 0 "C11" V 4400 3500 40  0000 L CNN
 F 1 "4.7" V 4650 3500 40  0000 L CNN
 F 2 "Capacitors_SMD:C_0805" H 4538 3400 30  0001 C CNN
@@
 $EndComp
 $Comp
-L C-RESCUE-BMS C?
+L C-RESCUE-BMS C9
 U 1 1 55DF2F5C
 P 4500 1900
-AR Path="/55BB8FBC/55844E2F/55DF2F5C" Ref="C?"  Part="1"
-AR Path="/55C14E4B/55844E2F/55DF2F5C" Ref="C?"  Part="1"
-AR Path="/55DF2F5C" Ref="C?"  Part="1"
-AR Path="/55844E2F/55DF2F5C" Ref="C1"  Part="1"
-F 0 "C1" V 4350 1850 40  0000 L CNN
+F 0 "C9" V 4350 1850 40  0000 L CNN
 F 1 "4.7" V 4650 1850 40  0000 L CNN
 F 2 "Capacitors_SMD:C_0805" H 4538 1750 30  0001 C CNN
