File: design/BQ/BQ.kicad_pcb (KiCad board)
At the start: 2 copper layers, 162 parts, among them K1 XLR3, Q1 BST82,215, Q10 MOSFET_N, Q11 MOSFET_N, Q12 DMN2300UFB4-7B, Q13 MOSFET_N, Q14 MOSFET_N, Q15 MOSFET_N, Q16 MOSFET_N, Q2 MOSFET_N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

Commit message: Add datasheets
Parts:
- removed C27, C28: 10u, Capacitors_SMD:C_0805
- added C24: 10u, Capacitors_SMD:C_0805, F.Cu at (90.0, 82.2)
- added C25: 10u, Capacitors_SMD:C_0805, F.Cu at (97.2, 84.2)
- C1, C12, C13, C14, C6, Cf2, Cf3, D18, D20, D22, D4, Q2, Q4, R1, R16, R17, R18, R22, R23, R24, R4: moved to B.Cu
- C10: value 4,7 -> 4.7; moved to B.Cu
- C11: value 0.1u -> 4.7; moved to B.Cu
- C2: value 4.7 -> 1u
- C3: value 4.7 -> 0.1u; moved to B.Cu
- C4: value 4.7 -> 1u; moved to B.Cu
- C7: value 1u -> 4,7
- C8: value 1u -> 0.1u; moved to B.Cu
- C9: value 0.1u -> 4.7
- K1: footprint Wire_Pads:SolderWirePad_2x_2mmDrill -> JSTcon:b2b-ph-kl
- Q1: footprint Transistors_SMD:sc70 -> CRF1:sc70; moved to B.Cu
- R10, R11, R12, R7: footprint Resistors_SMD:R_0805 -> Connect:PINHEAD1-2
- moved C21 134.8 mm to (276.4, 62.6)
- moved R54 134.0 mm to (268.9, 46.3)
- moved D32 132.0 mm to (269.6, 52.5)
- moved R60 131.1 mm to (272.6, 62.6)
- moved R56 130.7 mm to (265.3, 46.3)
- moved R55 128.0 mm to (265.3, 52.6)
- moved R61 127.7 mm to (268.9, 62.6)
- moved D34 126.4 mm to (269.6, 68.8)
- moved Q14 124.7 mm to (259.4, 48.0)
- moved R63 124.2 mm to (265.3, 62.6)
- moved R14 123.2 mm to (38.5, 49.5), turned to 270 degrees
- moved R62 122.2 mm to (265.3, 68.9)
- moved Cc2 119.4 mm to (267.5, 95.1)
- moved Q16 118.2 mm to (259.4, 64.3)
- moved Cc3 115.3 mm to (263.4, 95.1)
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Connections:
- C1 pad 1: -BATT_In -> /Vcc
- C1 pad 2: /NTC Temp monitor/Temp1_in -> -BATT_In
- C10 pad 1: -BATT_In -> /Battery_pack/B
- C10 pad 2: Net-(C10-Pad2) -> /NTC Temp monitor/Temp3_in
- C11 pad 1: Net-(C11-Pad1) -> /Battery_pack/A
- C11 pad 2: -BATT_In -> /NTC Temp monitor/Temp2_in
- C12 pad 1: /Battery_pack/VC4 -> /Battery_pack/VC1
- C12 pad 2: /Battery_pack/VC5 -> /Battery_pack/VC2
- C13 pad 1: /Battery_pack/A -> /Battery_pack/VC2
- C13 pad 2: /Battery_pack/VC6 -> /Battery_pack/VC3
- C14 pad 1: -BATT_In -> /Battery_pack/VC3
- C14 pad 2: /Battery_pack/VC1 -> /Battery_pack/VC4
- C15 pad 1: /Battery_pack/VC1 -> /Battery_pack/VC4
- C15 pad 2: /Battery_pack/VC2 -> /Battery_pack/VC5
- C16 pad 1: /Battery_pack/VC2 -> /Battery_pack/VC6
- C16 pad 2: /Battery_pack/VC3 -> /Battery_pack/VC7
- C17 pad 1: /Battery_pack/VC3 -> /Battery_pack/A
- C17 pad 2: /Battery_pack/VC4 -> /Battery_pack/VC6
- C18 pad 1: /Battery_pack/VC9 -> -BATT_In
- C18 pad 2: /Battery_pack/VC10 -> /Battery_pack/VC1
- C19 pad 1: /Battery_pack/VC6 -> /Battery_pack/VC7
- C19 pad 2: /Battery_pack/VC7 -> /Battery_pack/VC8
- C2 pad 1: /Battery_pack/B -> Net-(C2-Pad1)
- C2 pad 2: /NTC Temp monitor/Temp3_in -> -BATT_In
- C20 pad 1: /Battery_pack/BatteryVC10B-11/VC0_cap -> /Battery_pack/VC8
- C20 pad 2: /Battery_pack/VC11 -> /Battery_pack/VC9
- C21 pad 1: /Battery_pack/VC14 -> /Battery_pack/VC9
- C21 pad 2: /Battery_pack/VC15 -> /Battery_pack/VC10
- C22 pad 1: /Battery_pack/VC7 -> /Battery_pack/BatteryVC10B-11/VC0_cap
- C22 pad 2: /Battery_pack/VC8 -> /Battery_pack/VC11
- C23 pad 1: /Battery_pack/VC8 -> /Battery_pack/VC11
- C23 pad 2: /Battery_pack/VC9 -> /Battery_pack/VC12
- C26 pad 1: /Battery_pack/VC11 -> /Battery_pack/VC14
- C26 pad 2: /Battery_pack/VC12 -> /Battery_pack/VC15
- C3 pad 1: /Battery_pack/A -> Net-(C3-Pad1)
- C3 pad 2: /NTC Temp monitor/Temp2_in -> -BATT_In
- C4 pad 1: /Vcc -> /Battery_pack/A
- C4 pad 2: -BATT_In -> Net-(C4-Pad2)
- C5 pad 1: Net-(C5-Pad1) -> /Battery_pack/B
- C5 pad 2: -BATT_In -> Net-(C5-Pad2)
- C6 pad 2: -BATT_In -> Net-(C3-Pad1)
- C7 pad 1: /Battery_pack/A -> -BATT_In
- C8 pad 1: /Battery_pack/B -> Net-(C6-Pad1)
- C8 pad 2: Net-(C8-Pad2) -> -BATT_In
- C9 pad 1: Net-(C11-Pad1) -> -BATT_In
- C9 pad 2: Net-(C6-Pad1) -> /NTC Temp monitor/Temp1_in
- R16 pad 2: (no net) -> Net-(Q2-PadS)
- R19 pad 2: (no net) -> Net-(Q3-PadS)
- R22 pad 2: (no net) -> Net-(Q4-PadS)
- R26 pad 2: (no net) -> Net-(Q5-PadS)
- R29 pad 2: (no net) -> Net-(Q6-PadS)
- R32 pad 2: (no net) -> Net-(Q7-PadS)
- R35 pad 2: (no net) -> Net-(Q8-PadS)
- R38 pad 2: (no net) -> Net-(Q9-PadS)
- R41 pad 2: (no net) -> Net-(Q10-PadS)
- R45 pad 2: (no net) -> Net-(Q11-PadS)
- R48 pad 2: (no net) -> Net-(Q12-PadS)
- R5 pad 1: Net-(C6-Pad1) -> Net-(C3-Pad1)
- R51 pad 2: (no net) -> Net-(Q13-PadS)
- R54 pad 2: (no net) -> Net-(Q14-PadS)
- R57 pad 2: (no net) -> Net-(Q15-PadS)
- R6 pad 2: Net-(C10-Pad2) -> Net-(C7-Pad2)
- R61 pad 2: (no net) -> Net-(Q16-PadS)
- R8 pad 1: Net-(C11-Pad1) -> Net-(C6-Pad1)
- U1 pad 1: (no net) -> /DSG
- U1 pad 11: Net-(C7-Pad2) -> Net-(C4-Pad2)
- U1 pad 12: Net-(C7-Pad2) -> Net-(C4-Pad2)
- U1 pad 14: Net-(C7-Pad2) -> Net-(C4-Pad2)
- U1 pad 16: Net-(C8-Pad2) -> Net-(C5-Pad2)
- U1 pad 17: Net-(C8-Pad2) -> Net-(C5-Pad2)
- U1 pad 19: Net-(C8-Pad2) -> Net-(C5-Pad2)
- U1 pad 42: Net-(C6-Pad1) -> Net-(C3-Pad1)
- U1 pad 43: Net-(C11-Pad1) -> Net-(C6-Pad1)
- U1 pad 7: Net-(C5-Pad1) -> Net-(C2-Pad1)
- U1 pad 9: Net-(C10-Pad2) -> Net-(C7-Pad2)
Other:
- board outline added: 96.5 x 25.4 mm

Commit message: Start autorouting and palcing a components
Parts:
- moved C16 2.58 mm to (212.3, 33.4)
Changed lines of the file:
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@@
   )
   (module Capacitors_SMD:C_0805 (layer F.Cu)
-    (at 209.7 33.4)
+    (at 212.28 33.41)
     (descr "Capacitor SMD 0805, reflow soldering, AVX (see smccp.pdf)")
     (tags "capacitor 0805")
